File: BMI088.kicad_sch (KiCad schematic)
At the start: 1 part, among them U2 BMI088

Commit message: computer
Connections:
- net ACCEL_INT: no longer names the net of U2.16 (INT1)
- net GYRO_INT: no longer names the net of U2.12 (INT3)
- no-connect marks 2 -> 4
Changed lines of the file:
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@@
+	)
+	(no_connect
+		(at 157.48 104.14)
+	)
+	(no_connect
+		(at 157.48 99.06)
 	)
 	(no_connect
@@
 		)
 	)
-	(hierarchical_label "GYRO_INT"
-		(shape input)
-		(at 157.48 104.14 0)
-		(fields_autoplaced yes)
-		(effects
-			(font
-				(size 1.27 1.27)
-			)
-			(justify left)
-		)
-	)
 	(hierarchical_label "SDO_GYRO"
 		(shape input)
@@
 		)
 	)
-	(hierarchical_label "ACCEL_INT"
-		(shape input)
-		(at 157.48 99.06 0)
-		(fields_autoplaced yes)
-		(effects
-			(font
-				(size 1.27 1.27)
-			)
-			(justify left)
-		)
-	)
