File: NDXPCOMPUTER.kicad_pcb (KiCad board)
At the start: 2 copper layers, 31.4 x 55.6 mm, 71 parts, among them J10 Conn_02x06_Counter_Clockwise, J11 Conn_01x06, J2 USB_C_Receptacle_USB2.0_16P, J3 Conn_Coaxial, J4 Conn_02x10_Counter_Clockwise, J9 Conn_01x01, Q1 SSM3J328R, Q2 L2N7002SLLT1G, Q3 SSM3J328R, Q4 L2N7002SLLT1G, Q5 SSM3J328R, Q6 L2N7002SLLT1G, Q7 SSM3J328R, Q8 L2N7002SLLT1G, SW1 SW_Push, SW2 SW_Push, U1 STM32H723VGTx, U10 SP3485EN, U11 Ai-Thinker-Ra-01, U2 BMI088, U3 LSM6DSM, U4 BMP581, U5 NEO-M9N, U7 AP63203WU, U9 TPS62130

Commit message: routed🛣️
Parts:
- removed J4: Conn_02x10_Counter_Clockwise, Connector_PinSocket_2.54mm:PinSocket_2x10_P2.54mm_Vertical
- added J12: Conn_02x08_Counter_Clockwise, Connector_PinSocket_2.54mm:PinSocket_2x08_P2.54mm_Vertical, F.Cu at (153.8, 87.5)
- added J8: Micro_SD_Card, Connector_Card:microSD_HC_Wuerth_693072010801, F.Cu at (8.11, 7.37)
- U11: moved to B.Cu
- moved U11 56.0 mm to (140.8, 88.0), turned to 180 degrees
- moved J10 6.06 mm to (129.2, 105.3)
- moved J11 3.16 mm to (128.5, 87.6)
Connections:
- U1 pad 30: unconnected-(U1-PA6-Pad30) -> /BMP581/SDO_BARO
- U1 pad 31: unconnected-(U1-PA7-Pad31) -> /BMP581/SDI_BARO
- U1 pad 32: unconnected-(U1-PC4-Pad32) -> /BMP581/CS_BARO
- U1 pad 41: unconnected-(U1-PE11-Pad41) -> /LSM6DSM/CS_IMU_LOW
- U1 pad 42: unconnected-(U1-PE12-Pad42) -> /LSM6DSM/SCL_IMU_LOW
- U1 pad 43: unconnected-(U1-PE13-Pad43) -> /LSM6DSM/SDO_IMU_LOW
- U1 pad 44: unconnected-(U1-PE14-Pad44) -> /LSM6DSM/SDI_IMU_LOW
- U1 pad 59: unconnected-(U1-PD12-Pad59) -> /BMM350/SCK_MAG
- U1 pad 60: unconnected-(U1-PD13-Pad60) -> /BMM350/SDA_MAG
- U1 pad 80: unconnected-(U1-PC12-Pad80) -> /BMP581/SCK_BARO
- U3 pad 4: /LSM6DSM/INT_IMU_LOW -> unconnected-(U3-INT1-Pad4)
- U4 pad 7: /BMP581/INT_BARO -> unconnected-(U4-INT-Pad7)

Commit message: branches
Parts:
- removed C1, C18: 0.1uF, Capacitor_SMD:C_0402_1005Metric
- removed C10: 4.7uF, Capacitor_SMD:C_0603_1608Metric
- removed C11, C12: 2.2uF, Capacitor_SMD:C_0603_1608Metric
- removed C13, C21: 10uF, Capacitor_SMD:C_0805_2012Metric
- removed C14, C2, C3, C4, C5, C6, C7, C8, C9: 100nF, Capacitor_SMD:C_0402_1005Metric
- removed C15, C16, C20: 22uF, Capacitor_SMD:C_1206_3216Metric
- removed C17: 2.2uF, Capacitor_SMD:C_0402_1005Metric
- removed C19: 3.3nF, Capacitor_SMD:C_0402_1005Metric
- removed D1: D, Diode_SMD:D_SOD-323
- removed J10: Conn_02x06_Counter_Clockwise, Connector_PinHeader_2.54mm:PinHeader_2x06_P2.54mm_Vertical_SMD
- removed J8: Micro_SD_Card, Connector_Card:microSD_HC_Wuerth_693072010801
- removed J9: Conn_01x01, TestPoint:TestPoint_THTPad_D3.0mm_Drill1.5mm
- removed L1: 4.7uH, Inductor_SMD:L_1008_2520Metric
- removed L2: 2.2uH, Inductor_SMD:L_1008_2520Metric
- removed Q1, Q3, Q5, Q7: SSM3J328R, SSM3J328R:SOT95P240X88-3N
- removed Q2, Q4, Q6, Q8: L2N7002SLLT1G, Package_TO_SOT_SMD:SOT-23
- removed R1, R2: 5.1k, Resistor_SMD:R_0402_1005Metric
- removed R10, R13, R14, R15, R16, R4, R5, R8, R9: 100k, Resistor_SMD:R_0603_1608Metric
- removed R11: 1M, Resistor_SMD:R_0603_1608Metric
- removed R12: 200k, Resistor_SMD:R_0603_1608Metric
- removed R3: 10k, Resistor_SMD:R_0402_1005Metric
- removed R6, R7: 22, Resistor_SMD:R_0603_1608Metric
- removed SW1, SW2: SW_Push, Button_Switch_SMD:SW_SPST_B3U-1000P
- removed U10: SP3485EN, Package_SO:SOIC-8_3.9x4.9mm_P1.27mm
- removed U7: AP63203WU, Package_TO_SOT_SMD:TSOT-23-6
- removed U9: TPS62130, Package_DFN_QFN:VQFN-16-1EP_3x3mm_P0.5mm_EP1.68x1.68mm_ThermalVias
- added J13: Conn_02x06_Odd_Even, Connector_PinHeader_2.54mm:PinHeader_2x06_P2.54mm_Vertical_SMD, B.Cu at (129.0, 105.5)
Connections:
- net /BMM350/SCK_MAG renamed /STM32H7/SCK_MAG
- net /BMM350/SDA_MAG renamed /STM32H7/SDA_MAG
- J11 pad 1: unconnected-(J11-Pin_1-Pad1) -> USB_VBUS
- J11 pad 2: unconnected-(J11-Pin_2-Pad2) -> /Peripherals/TX_RFD900x
- J11 pad 3: unconnected-(J11-Pin_3-Pad3) -> /Peripherals/RX_RFD900x
- J11 pad 6: unconnected-(J11-Pin_6-Pad6) -> GND
- U1 pad 1: unconnected-(U1-PE2-Pad1) -> /Peripherals/PYRO_1
- U1 pad 2: unconnected-(U1-PE3-Pad2) -> /Peripherals/PYRO_2
- U1 pad 3: unconnected-(U1-PE4-Pad3) -> /Peripherals/PYRO_3
- U1 pad 4: unconnected-(U1-PE5-Pad4) -> /Peripherals/PYRO_4
- U1 pad 63: unconnected-(U1-PC6-Pad63) -> /RS485/TX_RS485
- U1 pad 64: unconnected-(U1-PC7-Pad64) -> /RS485/RX_RS485
- U1 pad 65: unconnected-(U1-PC8-Pad65) -> /RS485/DIR_RS485
- U1 pad 81: unconnected-(U1-PD0-Pad81) -> /LoRa/RST_LORA
- U1 pad 84: unconnected-(U1-PD3-Pad84) -> /LoRa/CS_LORA
- U11 pad 12: unconnected-(U11-SCK-Pad12) -> /BMP581/SCK_BARO
- U11 pad 13: unconnected-(U11-MISO-Pad13) -> /BMP581/SDO_BARO
- U11 pad 14: unconnected-(U11-MOSI-Pad14) -> /BMP581/SDI_BARO
- U11 pad 15: unconnected-(U11-~{NSS}-Pad15) -> /LoRa/CS_LORA
- U11 pad 16: Net-(U11-GND-Pad16) -> GND
- U11 pad 2: Net-(U11-GND-Pad16) -> GND
- U11 pad 3: unconnected-(U11-VDD-Pad3) -> +3.3V
- U11 pad 4: unconnected-(U11-~{RESET}-Pad4) -> /LoRa/RST_LORA
- U11 pad 9: Net-(U11-GND-Pad16) -> GND
