File: NDXPCOMPUTER.kicad_sch (KiCad schematic)
At the start: 0 parts

Commit message: sensors📡
Other:
- added sheet Power (power.kicad_sch)
Changed lines of the file:
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@@
 		)
 		(property "Sheetname" "NEO-M9N"
-			(at 215.9 145.034 0)
+			(at 214.122 144.018 0)
 			(effects
 				(font
@@
 				(path "/880cd2ad-ee8a-45d0-bf92-2f93a861aac0"
 					(page "6")
+				)
+			)
+		)
+	)
+	(sheet
+		(at 82.55 40.64)
+		(size 25.4 22.86)
+		(stroke
+			(width 0.1524)
+			(type solid)
+		)
+		(fill
+			(color 0 0 0 0.0000)
+		)
+		(property "Sheetname" "Power"
+			(at 91.694 52.832 0)
+			(effects
+				(font
+					(size 1.27 1.27)
+				)
+				(justify left bottom)
+			)
+		)
+		(property "Sheetfile" "power.kicad_sch"
+			(at 82.55 64.0846 0)
+			(effects
+				(font
+					(size 1.27 1.27)
+				)
+				(justify left top)
+			)
+		)
+		(instances
+			(project "NDXPCOMPUTER"
+				(path "/880cd2ad-ee8a-45d0-bf92-2f93a861aac0"
+					(page "7")
 				)
 			)
@@
 		)
 		(property "Sheetname" "BMI088"
-			(at 214.122 39.624 0)
+			(at 214.122 38.1 0)
 			(effects
 				(font

Commit message: board🏄‍♂️
Other:
- sheet BMI088 ports: added ACCEL_INT, CS_ACCEL, CS_GYRO, GYRO_INT, SCK, SDI, SDO_ACCEL, SDO_GYRO; removed none
- sheet STM32H7 ports: added CS_GYRO, SCK_GYRO, SDI_GYRO, SDO_GYRO; removed none
Changed lines of the file:
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@@
 		(rev "1.0")
+	)
+	(wire
+		(pts
+			(xy 177.8 77.47) (xy 190.5 77.47)
+		)
+		(stroke
+			(width 0)
+			(type default)
+		)
+	)
+	(wire
+		(pts
+			(xy 195.58 85.09) (xy 195.58 34.29)
+		)
+		(stroke
+			(width 0)
+			(type default)
+		)
+	)
+	(wire
+		(pts
+			(xy 195.58 34.29) (xy 204.47 34.29)
+		)
+		(stroke
+			(width 0)
+			(type default)
+		)
+	)
+	(wire
+		(pts
+			(xy 190.5 22.86) (xy 204.47 22.86)
+		)
+		(stroke
+			(width 0)
+			(type default)
+		)
+	)
+	(wire
+		(pts
+			(xy 193.04 80.01) (xy 193.04 30.48)
+		)
+		(stroke
+			(width 0)
+			(type default)
+		)
+	)
+	(wire
+		(pts
+			(xy 198.12 82.55) (xy 198.12 41.91)
+		)
+		(stroke
+			(width 0)
+			(type default)
+		)
+	)
+	(wire
+		(pts
+			(xy 193.04 30.48) (xy 204.47 30.48)
+		)
+		(stroke
+			(width 0)
+			(type default)
+		)
+	)
+	(wire
+		(pts
+			(xy 198.12 41.91) (xy 204.47 41.91)
+		)
+		(stroke
+			(width 0)
+			(type default)
+		)
+	)
+	(wire
+		(pts
+			(xy 177.8 80.01) (xy 193.04 80.01)
+		)
+		(stroke
+			(width 0)
+			(type default)
+		)
+	)
+	(wire
+		(pts
+			(xy 190.5 22.86) (xy 190.5 77.47)
+		)
+		(stroke
+			(width 0)
+			(type default)
+		)
+	)
+	(wire
+		(pts
+			(xy 177.8 85.09) (xy 195.58 85.09)
+		)
+		(stroke
+			(width 0)
+			(type default)
+		)
+	)
+	(wire
+		(pts
+			(xy 177.8 82.55) (xy 198.12 82.55)
+		)
+		(stroke
+			(width 0)
+			(type default)
+		)
 	)
 	(text "Barometer"
@@
 	(text "Low-G IMU"
 		(exclude_from_sim no)
-		(at 213.36 56.896 0)
+		(at 213.614 57.912 0)
 		(effects
 			(font
@@
 	(text "High-G IMU"
 		(exclude_from_sim no)
-		(at 214.122 24.892 0)
+		(at 214.122 17.272 0)
 		(effects
 			(font
@@
 		)
 		(property "Sheetname" "BMP280"
-			(at 213.36 106.934 0)
+			(at 214.376 105.918 0)
 			(effects
 				(font
@@
 	)
 	(sheet
-		(at 204.47 26.67)
-		(size 27.94 22.86)
+		(at 204.47 19.05)
+		(size 27.94 33.02)
 		(stroke
 			(width 0.1524)
@@
 		)
 		(property "Sheetname" "BMI088"
-			(at 214.122 38.1 0)
+			(at 214.63 35.306 0)
 			(effects
 				(font
@@
 		)
 		(property "Sheetfile" "BMI088.kicad_sch"
-			(at 204.47 50.1146 0)
+			(at 203.962 53.086 0)
 			(effects
 				(font
@@
 				)
 				(justify left top)
+			)
+		)
+		(pin "CS_GYRO" input
+			(at 204.47 22.86 180)
+			(effects
+				(font
+					(size 1.27 1.27)
+				)
+				(justify left)
+			)
+		)
+		(pin "CS_ACCEL" input
+			(at 204.47 26.67 180)
+			(effects
+				(font
+					(size 1.27 1.27)
+				)
+				(justify left)
+			)
+		)
+		(pin "SCK" input
+			(at 204.47 30.48 180)
+			(effects
+				(font
+					(size 1.27 1.27)
+				)
+				(justify left)
+			)
+		)
+		(pin "SDI" input
+			(at 204.47 34.29 180)
+			(effects
+				(font
+					(size 1.27 1.27)
+				)
+				(justify left)
+			)
+		)
+		(pin "SDO_ACCEL" input
+			(at 204.47 38.1 180)
+			(effects
+				(font
+					(size 1.27 1.27)
+				)
+				(justify left)
+			)
+		)
+		(pin "SDO_GYRO" input
+			(at 204.47 41.91 180)
+			(effects
+				(font
+					(size 1.27 1.27)
+				)
+				(justify left)
+			)
+		)
+		(pin "ACCEL_INT" input
+			(at 204.47 45.72 180)
+			(effects
+				(font
+					(size 1.27 1.27)
+				)
+				(justify left)
+			)
+		)
+		(pin "GYRO_INT" input
+			(at 204.47 49.53 180)
+			(effects
+				(font
+					(size 1.27 1.27)
+				)
+				(justify left)
 			)
 		)
@@
 			)
 		)
+		(pin "CS_GYRO" input
+			(at 177.8 77.47 0)
+			(effects
+				(font
+					(size 1.27 1.27)
+				)
+				(justify right)
+			)
+		)
+		(pin "SCK_GYRO" input
+			(at 177.8 80.01 0)
+			(effects
+				(font
+					(size 1.27 1.27)
+				)
+				(justify right)
+			)
+		)
+		(pin "SDI_GYRO" input
+			(at 177.8 82.55 0)
+			(effects
+				(font
+					(size 1.27 1.27)
+				)
+				(justify right)
+			)
+		)
+		(pin "SDO_GYRO" input
+			(at 177.8 85.09 0)
+			(effects
+				(font
+					(size 1.27 1.27)
+				)
+				(justify right)
+			)
+		)
 		(instances
 			(project "NDXPCOMPUTER"
@@
 	)
 	(sheet
-		(at 204.47 58.42)
+		(at 204.47 59.69)
 		(size 27.94 22.86)
 		(stroke
@@
 		)
 		(property "Sheetname" "LSM6DSM"
-			(at 214.122 71.374 0)
+			(at 214.122 72.644 0)
 			(effects
 				(font
@@
 		)
 		(property "Sheetfile" "LSM6DSM.kicad_sch"
-			(at 204.47 81.8646 0)
-			(effects
-				(font
+			(at 204.47 83.1346 0)
+			(effects
+				(font
