File: NDXPCOMPUTER.kicad_sch (KiCad schematic)
At the start: 0 parts

Commit message: gps🌎
Other:
- added sheet Peripherals (Peripherals.kicad_sch)
- sheet NEO-M9N ports: added CLK_GPS, CS_GPS, DI_GPS, DO_GPS; removed none
- sheet STM32H7 ports: added CS_GPS, SCK_GPS, SDI_GPS, SDO_GPS; removed none
Changed lines of the file:
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@@
+	(wire
+		(pts
+			(xy 177.8 123.19) (xy 195.58 123.19)
+		)
+		(stroke
+			(width 0)
+			(type default)
+		)
+	)
+	(wire
+		(pts
+			(xy 177.8 120.65) (xy 198.12 120.65)
+		)
+		(stroke
+			(width 0)
+			(type default)
+		)
+	)
+	(wire
+		(pts
+			(xy 177.8 125.73) (xy 193.04 125.73)
+		)
+		(stroke
+			(width 0)
+			(type default)
+		)
+	)
 	(wire
 		(pts
@@
 	(wire
 		(pts
+			(xy 177.8 118.11) (xy 200.66 118.11)
+		)
+		(stroke
+			(width 0)
+			(type default)
+		)
+	)
+	(wire
+		(pts
 			(xy 193.04 30.48) (xy 204.47 30.48)
 		)
@@
 	(wire
 		(pts
+			(xy 198.12 137.16) (xy 207.01 137.16)
+		)
+		(stroke
+			(width 0)
+			(type default)
+		)
+	)
+	(wire
+		(pts
+			(xy 200.66 134.62) (xy 207.01 134.62)
+		)
+		(stroke
+			(width 0)
+			(type default)
+		)
+	)
+	(wire
+		(pts
+			(xy 193.04 125.73) (xy 193.04 142.24)
+		)
+		(stroke
+			(width 0)
+			(type default)
+		)
+	)
+	(wire
+		(pts
 			(xy 198.12 41.91) (xy 204.47 41.91)
 		)
@@
 	(wire
 		(pts
+			(xy 198.12 120.65) (xy 198.12 137.16)
+		)
+		(stroke
+			(width 0)
+			(type default)
+		)
+	)
+	(wire
+		(pts
+			(xy 200.66 118.11) (xy 200.66 134.62)
+		)
+		(stroke
+			(width 0)
+			(type default)
+		)
+	)
+	(wire
+		(pts
+			(xy 193.04 142.24) (xy 207.01 142.24)
+		)
+		(stroke
+			(width 0)
+			(type default)
+		)
+	)
+	(wire
+		(pts
 			(xy 177.8 80.01) (xy 193.04 80.01)
 		)
@@
 	(wire
 		(pts
+			(xy 195.58 139.7) (xy 207.01 139.7)
+		)
+		(stroke
+			(width 0)
+			(type default)
+		)
+	)
+	(wire
+		(pts
 			(xy 190.5 22.86) (xy 190.5 77.47)
+		)
+		(stroke
+			(width 0)
+			(type default)
+		)
+	)
+	(wire
+		(pts
+			(xy 195.58 123.19) (xy 195.58 139.7)
 		)
 		(stroke
@@
 	(sheet
 		(at 207.01 130.81)
-		(size 25.4 22.86)
+		(size 25.4 15.24)
 		(stroke
 			(width 0.1524)
@@
 		)
 		(property "Sheetname" "NEO-M9N"
-			(at 214.122 144.018 0)
+			(at 218.948 141.224 0)
 			(effects
 				(font
@@
 		)
 		(property "Sheetfile" "NEO-M9N.kicad_sch"
-			(at 207.01 154.2546 0)
+			(at 207.01 147.32 0)
 			(effects
 				(font
@@
 				)
 				(justify left top)
+			)
+		)
+		(pin "CS_GPS" input
+			(at 207.01 134.62 180)
+			(effects
+				(font
+					(size 1.27 1.27)
+				)
+				(justify left)
+			)
+		)
+		(pin "DO_GPS" input
+			(at 207.01 137.16 180)
+			(effects
+				(font
+					(size 1.27 1.27)
+				)
+				(justify left)
+			)
+		)
+		(pin "DI_GPS" input
+			(at 207.01 139.7 180)
+			(effects
+				(font
+					(size 1.27 1.27)
+				)
+				(justify left)
+			)
+		)
+		(pin "CLK_GPS" input
+			(at 207.01 142.24 180)
+			(effects
+				(font
+					(size 1.27 1.27)
+				)
+				(justify left)
 			)
 		)
@@
 	)
 	(sheet
+		(at 74.93 85.09)
+		(size 31.75 34.29)
+		(stroke
+			(width 0.1524)
+			(type solid)
+		)
+		(fill
+			(color 0 0 0 0.0000)
+		)
+		(property "Sheetname" "Peripherals"
+			(at 85.09 102.616 0)
+			(effects
+				(font
+					(size 1.27 1.27)
+				)
+				(justify left bottom)
+			)
+		)
+		(property "Sheetfile" "Peripherals.kicad_sch"
+			(at 74.93 119.9646 0)
+			(effects
+				(font
+					(size 1.27 1.27)
+				)
+				(justify left top)
+			)
+		)
+		(instances
+			(project "NDXPCOMPUTER"
+				(path "/880cd2ad-ee8a-45d0-bf92-2f93a861aac0"
+					(page "8")
+				)
+			)
+		)
+	)
+	(sheet
 		(at 204.47 19.05)
 		(size 27.94 33.02)
@@
 			(effects
 				(font
+					(size 1.27 1.27)
+				)
+				(justify right)
+			)
+		)
+		(pin "SDI_GPS" input
+			(at 177.8 120.65 0)
+			(effects
+				(font
+					(size 1.27 1.27)
+				)
+				(justify right)
+			)
+		)
+		(pin "SCK_GPS" input
+			(at 177.8 125.73 0)
+			(effects
+				(font
+					(size 1.27 1.27)
+				)
+				(justify right)
+			)
+		)
+		(pin "CS_GPS" input
+			(at 177.8 118.11 0)
+			(effects
+				(font
+					(size 1.27 1.27)
+				)
+				(justify right)
+			)
+		)
+		(pin "SDO_GPS" input
+			(at 177.8 123.19 0)
+			(effects
+				(font

Commit message: test
Changed lines of the file:
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@@
 	(text "MCU"
 		(exclude_from_sim no)
-		(at 139.954 72.39 0)
+		(at 141.478 72.136 0)
 		(effects
 			(font

Commit message: test
Other:
- sheet LSM6DSM ports: added CS_IMU_LOW, INT_IMU_LOW, SCL_IMU_LOW, SDI_IMU_LOW, SDO_IMU_LOW; removed none
Changed lines of the file:
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@@
 		)
 		(property "Sheetname" "LSM6DSM"
-			(at 213.614 71.374 0)
+			(at 218.694 70.358 0)
 			(effects
 				(font
@@
 			)
 		)
+		(pin "SDI_IMU_LOW" input
+			(at 204.47 63.5 180)
+			(effects
+				(font
+					(size 1.27 1.27)
+				)
+				(justify left)
+			)
+		)
+		(pin "SDO_IMU_LOW" input
+			(at 204.47 66.04 180)
+			(effects
+				(font
+					(size 1.27 1.27)
+				)
+				(justify left)
+			)
+		)
+		(pin "SCL_IMU_LOW" input
+			(at 204.47 74.93 180)
+			(effects
+				(font
+					(size 1.27 1.27)
+				)
+				(justify left)
+			)
+		)
+		(pin "CS_IMU_LOW" input
+			(at 204.47 77.47 180)
+			(effects
+				(font
+					(size 1.27 1.27)
+				)
+				(justify left)
+			)
+		)
+		(pin "INT_IMU_LOW" input
+			(at 204.47 72.39 180)
+			(effects
+				(font
+					(size 1.27 1.27)
+				)
+				(justify left)
+			)
+		)

Commit message: Magnetometer🧲
Other:
- sheet BMP280 renamed BMP581
- added sheet BMM350 (BMM350.kicad_sch)
- sheet BMP581 ports: added CS_BARO, INT_BARO, SCK_BARO, SDI_BARO, SDO_BARO; removed none
- note added: "Magnetometer"
Changed lines of the file:
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@@
+		)
+	)
+	(text "Magnetometer"
+		(exclude_from_sim no)
+		(at 146.05 141.478 0)
+		(effects
+			(font
+				(size 2.032 2.032)
+			)
 		)
 	)
@@
 			(color 0 0 0 0.0000)
 		)
-		(property "Sheetname" "BMP280"
-			(at 214.376 105.918 0)
+		(property "Sheetname" "BMP581"
+			(at 214.63 106.426 0)
 			(effects
 				(font
@@
 			)
 		)
+		(pin "SDI_BARO" input
+			(at 208.28 96.52 180)
+			(effects
+				(font
+					(size 1.27 1.27)
+				)
+				(justify left)
+			)
+		)
+		(pin "SDO_BARO" input
+			(at 208.28 99.06 180)
+			(effects
+				(font
+					(size 1.27 1.27)
+				)
+				(justify left)
+			)
+		)
+		(pin "SCK_BARO" input
+			(at 208.28 101.6 180)
+			(effects
+				(font
+					(size 1.27 1.27)
+				)
+				(justify left)
+			)
+		)
+		(pin "CS_BARO" input
+			(at 208.28 109.22 180)
+			(effects
+				(font
+					(size 1.27 1.27)
+				)
+				(justify left)
+			)
+		)
+		(pin "INT_BARO" input
+			(at 208.28 111.76 180)
+			(effects
+				(font
+					(size 1.27 1.27)
+				)
+				(justify left)
+			)
+		)
 		(instances
 			(project "NDXPCOMPUTER"
@@
 				)
 			)
+		)
+	)
+	(sheet
+		(at 135.89 143.51)
+		(size 26.67 17.78)
+		(stroke
+			(width 0.1524)
+			(type solid)
+		)
+		(fill
+			(color 0 0 0 0.0000)
+		)
+		(property "Sheetname" "BMM350"
+			(at 144.272 153.162 0)
+			(effects
+				(font
+					(size 1.27 1.27)
+				)
+				(justify left bottom)
+			)
+		)
+		(property "Sheetfile" "BMM350.kicad_sch"
+			(at 135.89 161.8746 0)
+			(effects
+				(font
+					(size 1.27 1.27)
+				)
+				(justify left top)
+			)
+		)
+		(instances
+			(project "NDXPCOMPUTER"
+				(path "/880cd2ad-ee8a-45d0-bf92-2f93a861aac0"
+					(page "9")
+				)
+			)

Commit message: magnetic🧲
Other:
- sheet BMM350 ports: added INT_MAG, SCK_MAG, SDA_MAG; removed none
Changed lines of the file:
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@@
 	(text "Magnetometer"
 		(exclude_from_sim no)
-		(at 146.05 141.478 0)
+		(at 140.97 138.938 0)
 		(effects
 			(font
@@
 	)
 	(sheet
-		(at 135.89 143.51)
+		(at 130.81 142.24)
 		(size 26.67 17.78)
 		(stroke
@@
 		)
 		(property "Sheetname" "BMM350"
-			(at 144.272 153.162 0)
+			(at 139.192 151.892 0)
 			(effects
 				(font
@@
 		)
 		(property "Sheetfile" "BMM350.kicad_sch"
-			(at 135.89 161.8746 0)
-			(effects
-				(font
-					(size 1.27 1.27)
-				)
-				(justify left top)
-			)
-		)
+			(at 130.81 160.6046 0)
+			(effects
+				(font
+					(size 1.27 1.27)
+				)
+				(justify left top)
+			)
+		)
+		(pin "SCK_MAG" input
+			(at 157.48 146.05 0)
+			(effects
+				(font
+					(size 1.27 1.27)
+				)
+				(justify right)
+			)
+		)
+		(pin "SDA_MAG" input
+			(at 157.48 148.59 0)
+			(effects
+				(font
+					(size 1.27 1.27)
+				)
+				(justify right)
+			)
+		)
+		(pin "INT_MAG" input
+			(at 157.48 153.67 0)
+			(effects
+				(font
+					(size 1.27 1.27)
+				)
+				(justify right)
+			)
+		)

Commit message: 5v⚡️
Changed lines of the file:
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@@
 	(text "Magnetometer"
 		(exclude_from_sim no)
-		(at 140.97 138.938 0)
+		(at 140.716 139.7 0)
 		(effects
 			(font

Commit message: computer
Other:
- added sheet LoRa (LoRa.kicad_sch)
- added sheet RS485 (untitled.kicad_sch)
- added sheet SD (SD.kicad_sch)
- sheet BMI088 ports: added none; removed ACCEL_INT, GYRO_INT
- sheet STM32H7 ports: added CS_ACC, SCK_GYRO/ACC, SDI_GYRO/ACC, SDO_GYRO/ACC; removed CS_GPS, SCK_GPS, SCK_GYRO, SDI_GPS, SDI_GYRO, SDO_GPS, SDO_GYRO

Commit message: routed🛣️
Other:
- sheet BMM350 ports: added none; removed INT_MAG
- sheet BMP581 ports: added none; removed INT_BARO
- sheet LSM6DSM ports: added none; removed INT_IMU_LOW
- sheet Peripherals ports: added PYRO_1, PYRO_2, PYRO_3, PYRO_4; removed none
- sheet STM32H7 ports: added CS_BARO, CS_LOW_IMU, PYRO_1, PYRO_2, PYRO_3, PYRO_4, SCK_BARO, SCK_LOW_IMU, SCK_MAG, SDA_MAG, SDI_BARO, SDI_LOW_IMU, SDO_BARO, SDO_LOW_IMU; removed none
- note added: "Rework for UART"
