File: NDXPCOMPUTER.kicad_sch (KiCad schematic)
At the start: 0 parts

Commit message: branches
Other:
- sheet BMM350 ports: added SCL_MAG; removed SCK_MAG
- sheet LoRa ports: added CS_LORA, RST_LORA, SCK_LORA, SDI_LORA, SDO_LORA; removed none
- sheet RS485 ports: added DIR_RS485, RX_RS485, TX_RS485; removed none
- sheet STM32H7 ports: added CS_LORA, DIR_RS485, RST_LORA, RX_RS485, SCK_LORA, SDI_LORA, SDO_LORA, TX_RS485; removed none
- note added: "TODO: Rework for UART"
- note removed: "Rework for UART"
