File: _autosave-NDXPCOMPUTER.kicad_pcb (KiCad board)
At the start: 2 copper layers, 37 x 62.4 mm, 6 parts, among them P1 USB_C_Plug_USB2.0, U1 STM32H723VGTx, U2 BMI088, U3 LSM6DSM, U4 BMP280, U5 NEO-M9N

Commit message: usb-c🔌
Other:
- board size 37 x 62.4 mm -> 34.6 x 58.9 mm
Changed lines of the file:
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@@
 	(gr_rect
 		(start 122.2 66.45)
-		(end 159.2 128.85)
+		(end 156.8 125.35)
 		(stroke
 			(width 0.05)
