File: _autosave-NDXPCOMPUTER.kicad_pcb (KiCad board)
At the start: 2 copper layers, 31.4 x 55.6 mm, 71 parts, among them J10 Conn_02x06_Counter_Clockwise, J11 Conn_01x06, J2 USB_C_Receptacle_USB2.0_16P, J3 Conn_Coaxial, J4 Conn_02x10_Counter_Clockwise, J9 Conn_01x01, Q1 SSM3J328R, Q2 L2N7002SLLT1G, Q3 SSM3J328R, Q4 L2N7002SLLT1G, Q5 SSM3J328R, Q6 L2N7002SLLT1G, Q7 SSM3J328R, Q8 L2N7002SLLT1G, SW1 SW_Push, SW2 SW_Push, U1 STM32H723VGTx, U10 SP3485EN, U11 Ai-Thinker-Ra-01, U2 BMI088, U3 LSM6DSM, U4 BMP581, U5 NEO-M9N, U7 AP63203WU, U9 TPS62130

Commit message: LoRa🌊
Parts:
- U11: moved to B.Cu
- moved U11 56.0 mm to (140.8, 88.0), turned to 180 degrees
- moved J10 6.06 mm to (129.2, 105.3)
- moved J11 3.16 mm to (128.5, 87.6)
