File: NEO-M9N.kicad_sch (KiCad schematic)
At the start: 0 parts

Commit message: sensors📡
Parts:
- added U5: NEO-M9N, RF_GPS:ublox_NEO, symbol RF_GPS:NEO-M9N
Connections:
- new net: U5.10 (GND), U5.12 (GND), U5.13 (GND), U5.24 (GND)
Changed lines of the file:
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@@
 	(generator_version "8.0")
 	(paper "A4")
+	(symbol
+		(lib_id "RF_GPS:NEO-M9N")
+		(at 138.43 101.6 0)
+		(unit 1)
+		(exclude_from_sim no)
+		(in_bom yes)
+		(on_board yes)
+		(dnp no)
+		(fields_autoplaced yes)
+		(property "Reference" "U5"
+			(at 140.6241 124.46 0)
+			(effects
+				(font
+					(size 1.27 1.27)
+				)
+				(justify left)
+			)
+		)
+		(property "Value" "NEO-M9N"
+			(at 140.6241 127 0)
+			(effects
+				(font
+					(size 1.27 1.27)
+				)
+				(justify left)
+			)
+		)
+		(property "Footprint" "RF_GPS:ublox_NEO"
+			(at 148.59 123.19 0)
+			(effects
+				(font
+					(size 1.27 1.27)
+				)
+				(hide yes)
+			)
+		)
+		(property "Datasheet" "https://www.u-blox.com/sites/default/files/NEO-M9N-00B_DataSheet_UBX-19014285.pdf"
+			(at 138.43 101.6 0)
+			(effects
+				(font
+					(size 1.27 1.27)
+				)
+				(hide yes)
+			)
+		)
+		(property "Description" "GNSS Module NEO M8, VCC 2.7V to 3.6V"
+			(at 138.43 101.6 0)
+			(effects
+				(font
+					(size 1.27 1.27)
+				)
+				(hide yes)
+			)
+		)
+		(pin "10"
+		)
+		(pin "15"
+		)
+		(pin "17"
+		)
+		(pin "16"
+		)
+		(pin "1"
+		)
+		(pin "4"
+		)
+		(pin "5"
+		)
+		(pin "6"
+		)
+		(pin "7"
+		)
+		(pin "8"
+		)
+		(pin "9"
+		)
+		(pin "2"
+		)
+		(pin "20"
+		)
+		(pin "21"
+		)
+		(pin "22"
+		)
+		(pin "23"
+		)
+		(pin "24"
+		)
+		(pin "3"
+		)
+		(pin "12"
+		)
+		(pin "19"
+		)
+		(pin "18"
+		)
+		(pin "14"
+		)
+		(pin "11"
+		)
+		(pin "13"
+		)
+		(instances
+			(project ""
+				(path "/880cd2ad-ee8a-45d0-bf92-2f93a861aac0/16e7959a-598a-4fd4-86dd-9806303f6b27"
+					(reference "U5")
+					(unit 1)
+				)
+			)
+		)
+	)
 )

Commit message: gps🌎
Parts:
- added J3: Conn_Coaxial, Connector_Coaxial:U.FL_Hirose_U.FL-R-SMT-1_Vertical, symbol Connector:Conn_Coaxial
- added TP1: Safeboot, symbol Connector:TestPoint
Connections:
- net at U5.1 (~{SAFEBOOT}): now also TP1.1
- net GND: now reaches U5.10 (GND), U5.12 (GND), U5.13 (GND), U5.24 (GND)
- net GND: now also U5.2 (D_SEL), U5.7 (VDD_USB), J3.2 (Ext)
- net at U5.11 (RF_IN): now also J3.1 (In)
- net CS_GPS: now reaches U5.18 (SDA/~{SPI_CS})
- net CLK_GPS: now reaches U5.19 (SCL/SPI_CLK)
- net DO_GPS: now reaches U5.20 (TXD/SPI_MISO)
- net DI_GPS: now reaches U5.21 (RXD/SPI_MOSI)
- net +3.3V: now reaches U5.22 (V_BCKP)
- net +3.3V: now also U5.23 (VCC)
- no-connect marks 0 -> 6
Other:
- note added: "Low for spi"

Commit message: Magnetometer🧲
Parts:
- J3: footprint Connector_Coaxial:U.FL_Hirose_U.FL-R-SMT-1_Vertical -> Connector_Coaxial:SMA_Molex_73251-1153_EdgeMount_Horizontal
Changed lines of the file:
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@@
 			)
 		)
-		(property "Footprint" "Connector_Coaxial:U.FL_Hirose_U.FL-R-SMT-1_Vertical"
+		(property "Footprint" "Connector_Coaxial:SMA_Molex_73251-1153_EdgeMount_Horizontal"
 			(at 167.64 101.6 0)
 			(effects
