File: BMP280.kicad_sch (KiCad schematic)
At the start: 0 parts

Commit message: sensors📡
Parts:
- added U4: BMP280, Package_LGA:Bosch_LGA-8_2x2.5mm_P0.65mm_ClockwisePinNumbering, symbol Sensor_Pressure:BMP280
Changed lines of the file:
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@@
 	(generator_version "8.0")
 	(paper "A4")
+	(symbol
+		(lib_id "Sensor_Pressure:BMP280")
+		(at 135.89 107.95 0)
+		(unit 1)
+		(exclude_from_sim no)
+		(in_bom yes)
+		(on_board yes)
+		(dnp no)
+		(fields_autoplaced yes)
+		(property "Reference" "U4"
+			(at 142.24 105.4099 0)
+			(effects
+				(font
+					(size 1.27 1.27)
+				)
+				(justify left)
+			)
+		)
+		(property "Value" "BMP280"
+			(at 142.24 107.9499 0)
+			(effects
+				(font
+					(size 1.27 1.27)
+				)
+				(justify left)
+			)
+		)
+		(property "Footprint" "Package_LGA:Bosch_LGA-8_2x2.5mm_P0.65mm_ClockwisePinNumbering"
+			(at 135.89 125.73 0)
+			(effects
+				(font
+					(size 1.27 1.27)
+				)
+				(hide yes)
+			)
+		)
+		(property "Datasheet" "https://ae-bst.resource.bosch.com/media/_tech/media/datasheets/BST-BMP280-DS001.pdf"
+			(at 135.89 107.95 0)
+			(effects
+				(font
+					(size 1.27 1.27)
+				)
+				(hide yes)
+			)
+		)
+		(property "Description" "Absolute Barometric Pressure Sensor, LGA-8"
+			(at 135.89 107.95 0)
+			(effects
+				(font
+					(size 1.27 1.27)
+				)
+				(hide yes)
+			)
+		)
+		(pin "6"
+		)
+		(pin "8"
+		)
+		(pin "4"
+		)
+		(pin "5"
+		)
+		(pin "3"
+		)
+		(pin "7"
+		)
+		(pin "1"
+		)
+		(pin "2"
+		)
+		(instances
+			(project ""
+				(path "/880cd2ad-ee8a-45d0-bf92-2f93a861aac0/5e45f0a4-a72d-4462-856f-94f2b8339a46"
+					(reference "U4")
+					(unit 1)
+				)
+			)
+		)
+	)
 )

Commit message: usb-c🔌
Other:
- moved on the sheet: U4
Changed lines of the file:
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@@
 	(symbol
 		(lib_id "Sensor_Pressure:BMP280")
-		(at 135.89 107.95 0)
+		(at 146.05 105.41 0)
 		(unit 1)
 		(exclude_from_sim no)
@@
 		(fields_autoplaced yes)
 		(property "Reference" "U4"
-			(at 142.24 105.4099 0)
+			(at 152.4 102.8699 0)
 			(effects
 				(font
@@
 		)
 		(property "Value" "BMP280"
-			(at 142.24 107.9499 0)
+			(at 152.4 105.4099 0)
 			(effects
 				(font
@@
 		)
 		(property "Footprint" "Package_LGA:Bosch_LGA-8_2x2.5mm_P0.65mm_ClockwisePinNumbering"
-			(at 135.89 125.73 0)
+			(at 146.05 123.19 0)
 			(effects
 				(font
@@
 		)
 		(property "Datasheet" "https://ae-bst.resource.bosch.com/media/_tech/media/datasheets/BST-BMP280-DS001.pdf"
-			(at 135.89 107.95 0)
+			(at 146.05 105.41 0)
 			(effects
 				(font
@@
 		)
 		(property "Description" "Absolute Barometric Pressure Sensor, LGA-8"
-			(at 135.89 107.95 0)
+			(at 146.05 105.41 0)
 			(effects
 				(font

Commit message: Magnetometer🧲
Parts:
- removed U4: BMP280, Package_LGA:Bosch_LGA-8_2x2.5mm_P0.65mm_ClockwisePinNumbering, symbol Sensor_Pressure:BMP280
- added U4: BMP581, BMP581:BMP581, symbol BMP581:BMP581
Connections:
- new net +3.3V: U4.1 (VDDIO), U4.10 (VDD)
- new net CS_BARO: U4.6 (CSB)
- new net GND: U4.3 (GND), U4.8 (GND), U4.9 (GND)
- new net INT_BARO: U4.7 (INT)
- new net SCK_BARO: U4.2 (SCK/SCL)
- new net SDI_BARO: U4.4 (SDI/SDA)
- new net SDO_BARO: U4.5 (SDO/ADR)

Commit message: routed🛣️
Connections:
- net INT_BARO: no longer names the net of U4.7 (INT)
- no-connect marks 0 -> 1
Changed lines of the file:
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@@
 		(color 0 0 0 0)
+	)
+	(no_connect
+		(at 154.94 95.25)
 	)
 	(wire
@@
 		(fields_autoplaced yes)
 		(effects
-			(font
-				(size 1.27 1.27)
-			)
-			(justify left)
-		)
-	)
-	(hierarchical_label "INT_BARO"
-		(shape input)
-		(at 154.94 95.25 0)
-		(fields_autoplaced yes)
-		(effects
