File: LSM6DSM.kicad_sch (KiCad schematic)
At the start: 0 parts

Commit message: sensors📡
Parts:
- added U3: LSM6DSM, Package_LGA:LGA-14_3x2.5mm_P0.5mm_LayoutBorder3x4y, symbol Sensor_Motion:LSM6DSM
Connections:
- new net: U3.6 (GND), U3.7 (GND)
Changed lines of the file:
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@@
 	(generator_version "8.0")
 	(paper "A4")
+	(symbol
+		(lib_id "Sensor_Motion:LSM6DSM")
+		(at 142.24 97.79 0)
+		(unit 1)
+		(exclude_from_sim no)
+		(in_bom yes)
+		(on_board yes)
+		(dnp no)
+		(fields_autoplaced yes)
+		(property "Reference" "U3"
+			(at 144.4341 111.76 0)
+			(effects
+				(font
+					(size 1.27 1.27)
+				)
+				(justify left)
+			)
+		)
+		(property "Value" "LSM6DSM"
+			(at 144.4341 114.3 0)
+			(effects
+				(font
+					(size 1.27 1.27)
+				)
+				(justify left)
+			)
+		)
+		(property "Footprint" "Package_LGA:LGA-14_3x2.5mm_P0.5mm_LayoutBorder3x4y"
+			(at 132.08 115.57 0)
+			(effects
+				(font
+					(size 1.27 1.27)
+				)
+				(justify left)
+				(hide yes)
+			)
+		)
+		(property "Datasheet" "https://www.st.com/resource/en/datasheet/lsm6dsm.pdf"
+			(at 144.78 114.3 0)
+			(effects
+				(font
+					(size 1.27 1.27)
+				)
+				(hide yes)
+			)
+		)
+		(property "Description" "I2C/SPI, iNEMO inertial module: always-on 3D accelerometer and 3D gyroscope, with auxiliary SPI, 1.71V to 3.6V VCC"
+			(at 142.24 97.79 0)
+			(effects
+				(font
+					(size 1.27 1.27)
+				)
+				(hide yes)
+			)
+		)
+		(pin "7"
+		)
+		(pin "2"
+		)
+		(pin "10"
+		)
+		(pin "3"
+		)
+		(pin "13"
+		)
+		(pin "1"
+		)
+		(pin "5"
+		)
+		(pin "14"
+		)
+		(pin "11"
+		)
+		(pin "6"
+		)
+		(pin "8"
+		)
+		(pin "9"
+		)
+		(pin "4"
+		)
+		(pin "12"
+		)
+		(instances
+			(project ""
+				(path "/880cd2ad-ee8a-45d0-bf92-2f93a861aac0/f8f502cd-6130-4105-9076-c7ac7eb5037b"
+					(reference "U3")
+					(unit 1)
+				)
+			)
+		)
+	)
 )

Commit message: test
Connections:
- net SDO_IMU_LOW: now reaches U3.1 (SDO/SA0)
- net CS_IMU_LOW: now reaches U3.12 (CS)
- net SCL_IMU_LOW: now reaches U3.13 (SCL)
- net SDI_IMU_LOW: now reaches U3.14 (SDA)
- net GND: now reaches U3.2 (SDX)
- net GND: now also U3.3 (SCX), U3.6 (GND), U3.7 (GND)
- net INT_IMU_LOW: now reaches U3.4 (INT1)
- net +3.3V: now reaches U3.5 (VDDIO)
- net +3.3V: now also U3.8 (VDD)
- no-connect marks 0 -> 3

Commit message: routed🛣️
Connections:
- net INT_IMU_LOW: no longer names the net of U3.4 (INT1)
- no-connect marks 3 -> 4
Changed lines of the file:
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@@
 		(at 127 87.63)
+	)
+	(no_connect
+		(at 157.48 90.17)
 	)
 	(wire
@@
 		)
 	)
-	(hierarchical_label "INT_IMU_LOW"
-		(shape input)
-		(at 157.48 90.17 0)
-		(fields_autoplaced yes)
-		(effects
-			(font
-				(size 1.27 1.27)
-			)
-			(justify left)
-		)
-	)
