File: STM32H7.kicad_sch (KiCad schematic)
At the start: 1 part, among them U1 STM32H723VGTx

Commit message: board🏄‍♂️
Connections:
- net CS_GYRO: now reaches U1.28 (PA4)
- net SCK_GYRO: now reaches U1.29 (PA5)
- net SDI_GYRO: now reaches U1.30 (PA6)
- net SDO_GYRO: now reaches U1.31 (PA7)

Commit message: usb-c🔌
Parts:
- added D1: D, symbol Device:D
- added P1: USB_C_Plug_USB2.0, Connector_USB:USB_C_Receptacle_GCT_USB4105-xx-A_16P_TopMnt_Horizontal, symbol Connector:USB_C_Plug_USB2.0
- added R1: 5.1k, symbol Device:R
Connections:
- new net: D1.2 (A), P1.A4 (VBUS), P1.A9 (VBUS), P1.B4 (VBUS), P1.B9 (VBUS)
- new net: P1.A5 (CC), R1.2
- new net GND: P1.A1 (GND), P1.A12 (GND), P1.B1 (GND), P1.B12 (GND), P1.S1 (SHIELD), R1.1
- new net USB_VBUS: D1.1 (K)
- no-connect marks 0 -> 1

Commit message: mcu⚡️
Parts:
- removed P1: USB_C_Plug_USB2.0, Connector_USB:USB_C_Receptacle_GCT_USB4105-xx-A_16P_TopMnt_Horizontal, symbol Connector:USB_C_Plug_USB2.0
- added C1: C, symbol Device:C
- added J2: USB_C_Receptacle_USB2.0_16P, Connector_USB:USB_C_Receptacle_GCT_USB4105-xx-A_16P_TopMnt_Horizontal, symbol Connector:USB_C_Receptacle_USB2.0_16P
- added R2: 5.1k, symbol Device:R
- added R3: R, symbol Device:R
- added R6, R7: 22, symbol Device:R
- added SW1, SW2: SW_Push, Button_Switch_SMD:SW_SPST_B3U-1000P, symbol Switch:SW_Push
Connections:
- net CS_GYRO: no longer U1.28 (PA4)
- net GND: now also U1.10 (VSS), U1.19 (VSSA), U1.26 (VSS), U1.49 (VSS), U1.74 (VSS), U1.99 (VSS), C1.2, J2.A1 (GND), J2.A12 (GND), J2.B1 (GND), J2.B12 (GND), J2.S1 (SHIELD), R2.2, R3.2, SW2.1
- net SCK_GYRO: no longer U1.29 (PA5)
- net SDI_GYRO: now also U1.73 (VCAP); no longer U1.30 (PA6)
- net SDO_GYRO: now also U1.48 (VCAP); no longer U1.31 (PA7)
- net +3.3V: now reaches U1.100 (VDD)
- net +3.3V: now also U1.11 (VDD), U1.21 (VDDA), U1.27 (VDD), U1.50 (VDD), U1.6 (VBAT), U1.75 (VDD), SW1.1
- net at U1.14 (NRST): now also C1.1, SW2.2
- net at U1.69 (PA10): now also R7.1
- net at U1.70 (PA11): now also R6.1
- net at U1.94 (BOOT0): now also R3.1, SW1.2
- net at D1.2 (A): now also J2.A4 (VBUS), J2.A9 (VBUS), J2.B4 (VBUS), J2.B9 (VBUS)
- net at R1.2: now also J2.A5 (CC1)
- new net: J2.B5 (CC2), R2.1
- new net D+: J2.A6 (D+), J2.B6 (D+), R7.2
- new net D-: J2.A7 (D-), J2.B7 (D-), R6.2
- no-connect marks 1 -> 2
Other:
- note added: "route as differential pair, Resistors close to MCU"
- moved on the sheet: U1

Commit message: gps🌎
Parts:
- added C11, C12: C, 2.2uF, symbol Device:C
- R3: footprint (none) -> 10k
Connections:
- net +3.3V: now also U1.20 (VREF+)
- net CS_GYRO: now also U1.28 (PA4)
- net GND: now also U1.12 (PH0), C11.1, C12.1
- net SCK_GYRO: now also U1.29 (PA5)
- net SDI_GYRO: now also U1.30 (PA6); no longer U1.73 (VCAP)
- net SDO_GYRO: now also U1.31 (PA7); no longer U1.48 (VCAP)
- net CS_GPS: now reaches U1.41 (PE11)
- net SCK_GPS: now reaches U1.42 (PE12)
- net SDI_GPS: now reaches U1.43 (PE13)
- net SDO_GPS: now reaches U1.44 (PE14)
- new net: C11.2, U1.48 (VCAP)
- new net: C12.2, U1.73 (VCAP)
- no-connect marks 2 -> 3
Other:
- note added: "OSC_IN"
- note added: "route as differential pair, resistors close to MCU"
- note removed: "route as differential pair, Resistors close to MCU"

Commit message: test
Parts:
- C1: value C -> 0.1uF; footprint (none) -> Capacitor_SMD:C_0402_1005Metric
- C11, C12: value C -> 2.2uF; footprint 2.2uF -> Capacitor_SMD:C_0603_1608Metric
- D1: footprint (none) -> Diode_SMD:D_SOD-323
Other:
- moved on the sheet: C1

Commit message: FETS🦈
Parts:
- R1, R2: footprint (none) -> Resistor_SMD:R_0402_1005Metric
- R3: value R -> 10k; footprint 10k -> Resistor_SMD:R_0402_1005Metric
- R6, R7: footprint (none) -> Resistor_SMD:R_0603_1608Metric

Commit message: computer
Connections:
- net CS_GYRO: now also U1.77 (PA15(JTDI)); no longer U1.28 (PA4)
- net at R7.1: now also U1.71 (PA12); no longer U1.69 (PA10)
- net SDO_GYRO/ACC: now reaches U1.36 (PB2)
- net CS_ACC: now reaches U1.76 (PA14(JTCK)
- net SCK_GYRO/ACC: now reaches U1.78 (PC10)
- net SDI_GYRO/ACC: now reaches U1.79 (PC11)
- net CS_GPS: no longer names the net of U1.41 (PE11)
- net SCK_GPS: no longer names the net of U1.42 (PE12)
- net SCK_GYRO: no longer names the net of U1.29 (PA5)
- net SDI_GPS: no longer names the net of U1.43 (PE13)
- net SDI_GYRO: no longer names the net of U1.30 (PA6)
- net SDO_GPS: no longer names the net of U1.44 (PE14)
- net SDO_GYRO: no longer names the net of U1.31 (PA7)
Other:
- moved on the sheet: C1, C11, C12, D1, J2, R1, R2, R3, R6, R7, SW1, SW2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

Commit message: routed🛣️
Connections:
- net PYRO_1: now reaches U1.1 (PE2)
- net PYRO_2: now reaches U1.2 (PE3)
- net PYRO_3: now reaches U1.3 (PE4)
- net SDI_BARO: now reaches U1.30 (PA6)
- net SDO_BARO: now reaches U1.31 (PA7)
- net CS_BARO: now reaches U1.32 (PC4)
- net PYRO_4: now reaches U1.4 (PE5)
- net CS_LOW_IMU: now reaches U1.41 (PE11)
- net SCK_LOW_IMU: now reaches U1.42 (PE12)
- net SDI_LOW_IMU: now reaches U1.43 (PE13)
- net SDO_LOW_IMU: now reaches U1.44 (PE14)
- net SCK_MAG: now reaches U1.59 (PD12)
- net SDA_MAG: now reaches U1.60 (PD13)
- net SCK_BARO: now reaches U1.80 (PC12)
