File: STM32H7.kicad_sch (KiCad schematic)
At the start: 13 parts, among them J2 USB_C_Receptacle_USB2.0_16P, SW1 SW_Push, SW2 SW_Push, U1 STM32H723VGTx

Commit message: branches
Parts:
- added C10: 4.7uF, Capacitor_SMD:C_0603_1608Metric, symbol Device:C
- added C2, C3, C4, C5, C6, C7, C8, C9: 100nF, Capacitor_SMD:C_0402_1005Metric, symbol Device:C
- added JP1: SolderJumper_2_Open, Jumper:SolderJumper-2_P1.3mm_Open_TrianglePad1.0x1.5mm, symbol Jumper:SolderJumper_2_Open
Connections:
- net +3.3V: now also C10.1, C2.1, C3.1, C4.1, C5.1, C6.1, C7.1, C8.1, C9.1
- net GND: now also C10.2, C2.2, C3.2, C4.2, C5.2, C6.2, C7.2, C8.2, C9.2
- net at C1.1, SW2.2: now also JP1.1 (A); no longer U1.14 (NRST)
- net TX_RS485: now reaches U1.63 (PC6)
- net RX_RS485: now reaches U1.64 (PC7)
- net DIR_RS485: now reaches U1.65 (PC8)
- net RST_LORA: now reaches U1.81 (PD0)
- net CS_LORA: now reaches U1.84 (PD3)
- new net: JP1.2 (B), U1.14 (NRST)
Other:
- note added: "Decoupling for MCU 8 x 100nF, 1 x 4.7uF"
- moved on the sheet: C1, SW2
