File: BMM350.kicad_sch (KiCad schematic)
At the start: 1 part, among them U8 BMM350

Commit message: magnetic🧲
Parts:
- added C17: C, 2.2uF, symbol Device:C
Connections:
- net INT_MAG: now reaches U8.A1 (INT)
- net SDA_MAG: now reaches U8.A2 (SDA)
- net SCK_MAG: now reaches U8.A3 (SCK)
- net GND: now reaches U8.B1 (GND)
- net GND: now also U8.C3 (BYPASS), C17.2
- net +3.3V: now reaches U8.B2 (ADSEL)
- net +3.3V: now also U8.B3 (VDDIO), U8.C1 (VDD)
- net at U8.C2 (CRST): now also C17.1

Commit message: FETS🦈
Parts:
- C17: value C -> 2.2uF; footprint 2.2uF -> Capacitor_SMD:C_0402_1005Metric
Changed lines of the file:
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@@
 			)
 		)
-		(property "Value" "C"
+		(property "Value" "2.2uF"
 			(at 172.72 91.44 90)
 			(effects
@@
 			)
 		)
-		(property "Footprint" "2.2uF"
+		(property "Footprint" "Capacitor_SMD:C_0402_1005Metric"
 			(at 176.53 95.5548 0)
 			(effects

Commit message: routed🛣️
Connections:
- net INT_MAG: no longer names the net of U8.A1 (INT)
- no-connect marks 0 -> 1
Changed lines of the file:
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@@
 		(color 0 0 0 0)
+	)
+	(no_connect
+		(at 125.73 93.98)
 	)
 	(wire
@@
 		(fields_autoplaced yes)
 		(effects
-			(font
-				(size 1.27 1.27)
-			)
-			(justify right)
-		)
-	)
-	(hierarchical_label "INT_MAG"
-		(shape input)
-		(at 125.73 93.98 180)
-		(fields_autoplaced yes)
-		(effects

Commit message: branches
Parts:
- removed U8: BMM350, BGA9_BMM350_BOS, symbol BMM350:BMM350
- added C29, C30: 100nF, Capacitor_SMD:C_0402_1005Metric, symbol Device:C
- added C31: 10uF, Capacitor_SMD:C_0201_0603Metric, symbol Device:C
- added IC1: IIS2MDCTR, IIS2MDCTR:IIS2MDCTR, symbol IIS2MDCTR:IIS2MDCTR
- C17: value 2.2uF -> 220nF
Connections:
- net +3.3V: now also C29.1, C30.1, C31.1, IC1.10 (VDD_IO), IC1.3 (CS), IC1.9 (VDD)
- net GND: now also C29.2, C30.2, C31.2, IC1.6 (GND_1), IC1.8 (GND_2)
- net SDA_MAG: now also IC1.4 (SDA/SDI/SDO)
- net at C17.1: now also IC1.5 (C1)
- new net SCL_MAG: IC1.1 (SCL/SPC)
- no-connect marks 1 -> 4
