File: Peripherals.kicad_sch (KiCad schematic)
At the start: 5 parts, among them J1 Conn_01x02, Q1 PMOS, Q2 NMOS, U6 TPS62133

Commit message: Magnetometer🧲
Parts:
- added J4: Conn_02x10_Counter_Clockwise, Connector_PinSocket_2.54mm:PinSocket_2x10_P2.54mm_Vertical, symbol Connector_Generic:Conn_02x10_Counter_Clockwise
Changed lines of the file:
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@@
+	)
+	(symbol
+		(lib_id "Connector_Generic:Conn_02x10_Counter_Clockwise")
+		(at 214.63 120.65 0)
+		(unit 1)
+		(exclude_from_sim no)
+		(in_bom yes)
+		(on_board yes)
+		(dnp no)
+		(fields_autoplaced yes)
+		(property "Reference" "J4"
+			(at 215.9 104.14 0)
+			(effects
+				(font
+					(size 1.27 1.27)
+				)
+			)
+		)
+		(property "Value" "Conn_02x10_Counter_Clockwise"
+			(at 215.9 106.68 0)
+			(effects
+				(font
+					(size 1.27 1.27)
+				)
+			)
+		)
+		(property "Footprint" "Connector_PinSocket_2.54mm:PinSocket_2x10_P2.54mm_Vertical"
+			(at 214.63 120.65 0)
+			(effects
+				(font
+					(size 1.27 1.27)
+				)
+				(hide yes)
+			)
+		)
+		(property "Datasheet" "~"
+			(at 214.63 120.65 0)
+			(effects
+				(font
+					(size 1.27 1.27)
+				)
+				(hide yes)
+			)
+		)
+		(property "Description" "Generic connector, double row, 02x10, counter clockwise pin numbering scheme (similar to DIP package numbering), script generated (kicad-library-utils/schlib/autogen/connector/)"
+			(at 214.63 120.65 0)
+			(effects
+				(font
+					(size 1.27 1.27)
+				)
+				(hide yes)
+			)
+		)
+		(pin "10"
+		)
+		(pin "15"
+		)
+		(pin "5"
+		)
+		(pin "13"
+		)
+		(pin "9"
+		)
+		(pin "7"
+		)
+		(pin "4"
+		)
+		(pin "1"
+		)
+		(pin "8"
+		)
+		(pin "19"
+		)
+		(pin "20"
+		)
+		(pin "2"
+		)
+		(pin "3"
+		)
+		(pin "16"
+		)
+		(pin "11"
+		)
+		(pin "12"
+		)
+		(pin "18"
+		)
+		(pin "14"
+		)
+		(pin "17"
+		)
+		(pin "6"
+		)
+		(instances
+			(project ""
+				(path "/880cd2ad-ee8a-45d0-bf92-2f93a861aac0/933c923e-9649-42a5-9bc4-db8878fb4adc"
+					(reference "J4")
+					(unit 1)
+				)
+			)
+		)
 	)
 	(symbol

Commit message: 5v⚡️
Parts:
- removed U6: TPS62133, Package_DFN_QFN:VQFN-16-1EP_3x3mm_P0.5mm_EP1.68x1.68mm_ThermalVias, symbol Regulator_Switching:TPS62133
- added J5, J6, J7: Conn_01x02, symbol Connector_Generic:Conn_01x02
- added Q3, Q5, Q7: PMOS, symbol Simulation_SPICE:PMOS
- added Q4, Q6, Q8: NMOS, symbol Simulation_SPICE:NMOS
- added R5, R8, R9: R, 10k, symbol Device:R
Connections:
- net +BATT: now also Q3.3 (S), Q5.3 (S), Q7.3 (S), R5.1, R8.1, R9.1
- net GND: now also J5.1 (Pin_1), J6.1 (Pin_1), J7.1 (Pin_1), Q4.3 (S), Q6.3 (S), Q8.3 (S)
- new net: Q5.2 (G), Q6.1 (D), R8.2
- new net: J5.2 (Pin_2), Q3.1 (D)
- new net: Q3.2 (G), Q4.1 (D), R5.2
- new net: J7.2 (Pin_2), Q7.1 (D)
- new net: Q7.2 (G), Q8.1 (D), R9.2
- new net: J6.2 (Pin_2), Q5.1 (D)
Other:
- note removed: "Use this for 5v pyro"
- moved on the sheet: J1, Q1, Q2, R4

Commit message: FETS🦈
Parts:
- added R13, R14, R15, R16: 100k, Resistor_SMD:R_0603_1608Metric, symbol Device:R
- Q1, Q3, Q5, Q7: value PMOS -> SSM3J328R; footprint (none) -> SSM3J328R:SOT95P240X88-3N
- Q2, Q4, Q6, Q8: value NMOS -> L2N7002SLLT1G; footprint (none) -> Package_TO_SOT_SMD:SOT-23
- R4, R5, R8, R9: value R -> 100k; footprint 10k -> Resistor_SMD:R_0603_1608Metric
Connections:
- net +BATT: now also R15.1; no longer R8.1
- net at Q3.2 (G), R5.2: now also R8.1; no longer Q4.1 (D)
- net at Q1.2 (G), R4.2: now also R13.1; no longer Q2.1 (D)
- new net: Q5.2 (G), R14.1, R9.2
- new net: Q4.1 (D), R8.2
- new net: Q6.1 (D), R14.2
- new net: Q2.1 (D), R13.2
- new net: Q7.2 (G), R15.2, R16.1
- new net: Q8.1 (D), R16.2
Other:
- note added: "Found this pmos by digikey, 20v, in stock, pmos, scrolling for high amperage"
- note added: "SSM3J328R PMOS"
- note removed: "SK2301AA PMOS"
- moved on the sheet: J1, Q2

Commit message: computer
Other:
- note added: "Breakout Spare UARTS, 1x I2C, 1xSPI, 5v, 3v,"
- moved on the sheet: J4
Changed lines of the file:
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@@
 	)
 	(rectangle
-		(start 189.484 99.314)
-		(end 242.824 138.684)
+		(start 212.344 120.904)
+		(end 265.684 160.274)
 		(stroke
 			(width 0)
@@
 	)
 	(rectangle
-		(start 189.23 45.72)
-		(end 242.57 85.09)
+		(start 212.598 72.39)
+		(end 265.938 111.76)
 		(stroke
 			(width 0)
@@
 		)
 	)
+	(text "Breakout Spare UARTS, 1x I2C, 1xSPI, 5v, 3v, "
+		(exclude_from_sim no)
+		(at 259.588 118.364 0)
+		(effects
+			(font
+				(size 1.27 1.27)
+			)
+		)
+	)
 	(text "GPIO"
 		(exclude_from_sim no)
-		(at 191.77 97.79 0)
+		(at 214.63 119.38 0)
 		(effects
 			(font
@@
 	(text "PWM Output"
 		(exclude_from_sim no)
-		(at 195.072 44.45 0)
+		(at 218.44 71.12 0)
 		(effects
 			(font
@@
 	(symbol
 		(lib_id "Connector_Generic:Conn_02x10_Counter_Clockwise")
-		(at 214.63 120.65 0)
+		(at 237.49 142.24 0)
 		(unit 1)
 		(exclude_from_sim no)
@@
 		(fields_autoplaced yes)
 		(property "Reference" "J4"
-			(at 215.9 104.14 0)
+			(at 238.76 125.73 0)
 			(effects
 				(font
@@
 		)
 		(property "Value" "Conn_02x10_Counter_Clockwise"
-			(at 215.9 106.68 0)
+			(at 238.76 128.27 0)
 			(effects
 				(font
@@
 		)
 		(property "Footprint" "Connector_PinSocket_2.54mm:PinSocket_2x10_P2.54mm_Vertical"
-			(at 214.63 120.65 0)
+			(at 237.49 142.24 0)
 			(effects
 				(font
@@
 		)
 		(property "Datasheet" "~"
-			(at 214.63 120.65 0)
+			(at 237.49 142.24 0)
 			(effects
 				(font
@@
 		)
 		(property "Description" "Generic connector, double row, 02x10, counter clockwise pin numbering scheme (similar to DIP package numbering), script generated (kicad-library-utils/schlib/autogen/connector/)"
-			(at 214.63 120.65 0)
-			(effects
-				(font
+			(at 237.49 142.24 0)
+			(effects
+				(font

Commit message: LoRa🌊
Parts:
- added H1, H2, H3, H4: MountingHole, MountingHole:MountingHole_2.2mm_M2_DIN965_Pad, symbol Mechanical:MountingHole
- added J10: Conn_02x06_Counter_Clockwise, Connector_PinHeader_2.54mm:PinHeader_2x06_P2.54mm_Vertical_SMD, symbol Connector_Generic:Conn_02x06_Counter_Clockwise
- added J11: Conn_01x06, SM06B-GHS-TB:JST_SM06B-GHS-TB_LF__SN_, symbol Connector_Generic:Conn_01x06
Other:
- note added: "PWM/Servo Output"
- note added: "Power Pin Header"
- note added: "SM06B-GHS-TB(LF)(SN)"
- note added: "Telemetry Port (RFD900x)"
- note removed: "PWM Output"

Commit message: routed🛣️
Parts:
- removed J4: Conn_02x10_Counter_Clockwise, Connector_PinSocket_2.54mm:PinSocket_2x10_P2.54mm_Vertical, symbol Connector_Generic:Conn_02x10_Counter_Clockwise
- added J12: Conn_02x08_Counter_Clockwise, Connector_PinSocket_2.54mm:PinSocket_2x08_P2.54mm_Vertical, symbol Connector_Generic:Conn_02x08_Counter_Clockwise
Connections:
- net PYRO_2: now reaches Q4.2 (G)
- net PYRO_3: now reaches Q6.2 (G)
- net PYRO_1: now reaches Q2.2 (G)
- net PYRO_4: now reaches Q8.2 (G)
Changed lines of the file:
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@@
+	(wire
+		(pts
+			(xy 43.18 119.38) (xy 45.72 119.38)
+		)
+		(stroke
+			(width 0)
+			(type default)
+		)
+	)
 	(wire
 		(pts
@@
 	(wire
 		(pts
-			(xy 88.9 54.61) (xy 88.9 72.39)
+			(xy 86.36 54.61) (xy 86.36 72.39)
+		)
+		(stroke
+			(width 0)
+			(type default)
+		)
+	)
+	(wire
+		(pts
+			(xy 86.36 72.39) (xy 88.9 72.39)
 		)
 		(stroke
@@
 	(wire
 		(pts
-			(xy 45.72 101.6) (xy 45.72 119.38)
+			(xy 43.18 101.6) (xy 45.72 101.6)
+		)
+		(stroke
+			(width 0)
+			(type default)
+		)
+	)
+	(wire
+		(pts
+			(xy 87.63 120.65) (xy 90.17 120.65)
+		)
+		(stroke
+			(width 0)
+			(type default)
+		)
+	)
+	(wire
+		(pts
+			(xy 43.18 101.6) (xy 43.18 119.38)
 		)
 		(stroke
@@
 	(wire
 		(pts
+			(xy 43.18 53.34) (xy 45.72 53.34)
+		)
+		(stroke
+			(width 0)
+			(type default)
+		)
+	)
+	(wire
+		(pts
 			(xy 48.26 40.64) (xy 48.26 39.37)
 		)
@@
 	(wire
 		(pts
+			(xy 87.63 102.87) (xy 90.17 102.87)
+		)
+		(stroke
+			(width 0)
+			(type default)
+		)
+	)
+	(wire
+		(pts
+			(xy 43.18 71.12) (xy 45.72 71.12)
+		)
+		(stroke
+			(width 0)
+			(type default)
+		)
+	)
+	(wire
+		(pts
 			(xy 110.49 120.65) (xy 105.41 120.65)
 		)
@@
 	(wire
 		(pts
-			(xy 45.72 53.34) (xy 45.72 71.12)
+			(xy 43.18 53.34) (xy 43.18 71.12)
 		)
 		(stroke
@@
 	(wire
 		(pts
+			(xy 86.36 54.61) (xy 88.9 54.61)
+		)
+		(stroke
+			(width 0)
+			(type default)
+		)
+	)
+	(wire
+		(pts
 			(xy 45.72 43.18) (xy 48.26 43.18)
 		)
@@
 	(wire
 		(pts
-			(xy 90.17 102.87) (xy 90.17 120.65)
+			(xy 87.63 102.87) (xy 87.63 120.65)
 		)
 		(stroke
@@
 		)
 	)
+	(hierarchical_label "PYRO_2"
+		(shape input)
+		(at 96.52 63.5 180)
+		(fields_autoplaced yes)
+		(effects
+			(font
+				(size 1.27 1.27)
+			)
+			(justify right)
+		)
+	)
+	(hierarchical_label "PYRO_1"
+		(shape input)
+		(at 53.34 62.23 180)
+		(fields_autoplaced yes)
+		(effects
+			(font
+				(size 1.27 1.27)
+			)
+			(justify right)
+		)
+	)
+	(hierarchical_label "PYRO_4"
+		(shape input)
+		(at 97.79 111.76 180)
+		(fields_autoplaced yes)
+		(effects
+			(font
+				(size 1.27 1.27)
+			)
+			(justify right)
+		)
+	)
+	(hierarchical_label "PYRO_3"
+		(shape input)
+		(at 53.34 110.49 180)
+		(fields_autoplaced yes)
+		(effects
+			(font
+				(size 1.27 1.27)
+			)
+			(justify right)
+		)
+	)
 	(symbol
 		(lib_id "power:GND")
@@
 	)
 	(symbol
-		(lib_id "Connector_Generic:Conn_02x10_Counter_Clockwise")
-		(at 237.49 142.24 0)
-		(unit 1)
-		(exclude_from_sim no)
-		(in_bom yes)
-		(on_board yes)
-		(dnp no)
-		(fields_autoplaced yes)
-		(property "Reference" "J4"
-			(at 238.76 125.73 0)
-			(effects
-				(font
-					(size 1.27 1.27)
-				)
-			)
-		)
-		(property "Value" "Conn_02x10_Counter_Clockwise"
-			(at 238.76 128.27 0)
-			(effects
-				(font
-					(size 1.27 1.27)
-				)
-			)
-		)
-		(property "Footprint" "Connector_PinSocket_2.54mm:PinSocket_2x10_P2.54mm_Vertical"
-			(at 237.49 142.24 0)
-			(effects
-				(font
-					(size 1.27 1.27)
-				)
-				(hide yes)
-			)
-		)
-		(property "Datasheet" "~"
-			(at 237.49 142.24 0)
-			(effects
-				(font
-					(size 1.27 1.27)
-				)
-				(hide yes)
-			)
-		)
-		(property "Description" "Generic connector, double row, 02x10, counter clockwise pin numbering scheme (similar to DIP package numbering), script generated (kicad-library-utils/schlib/autogen/connector/)"
-			(at 237.49 142.24 0)
-			(effects
-				(font
-					(size 1.27 1.27)
-				)
-				(hide yes)
-			)
-		)
-		(pin "10"
-		)
-		(pin "15"
-		)
-		(pin "5"
-		)
-		(pin "13"
-		)
-		(pin "9"
-		)
-		(pin "7"
-		)
-		(pin "4"
-		)
-		(pin "1"
-		)
-		(pin "8"
-		)
-		(pin "19"
-		)
-		(pin "20"
-		)
-		(pin "2"
-		)
-		(pin "3"
-		)
-		(pin "16"
-		)
-		(pin "11"
-		)
-		(pin "12"
-		)
-		(pin "18"
-		)
-		(pin "14"
-		)
-		(pin "17"
-		)
-		(pin "6"
-		)
-		(instances
-			(project ""
-				(path "/880cd2ad-ee8a-45d0-bf92-2f93a861aac0/933c923e-9649-42a5-9bc4-db8878fb4adc"
-					(reference "J4")
-					(unit 1)
-				)
-			)
-		)
-	)
-	(symbol
 		(lib_id "power:GND")
 		(at 109.22 76.2 0)
@@
 					(unit 1)
 				)
+			)
+		)
+	)
+	(symbol
+		(lib_id "Connector_Generic:Conn_02x08_Counter_Clockwise")
+		(at 237.49 140.97 0)
+		(unit 1)
+		(exclude_from_sim no)
+		(in_bom yes)
+		(on_board yes)
+		(dnp no)
+		(fields_autoplaced yes)
+		(property "Reference" "J12"
+			(at 238.76 127 0)
+			(effects
+				(font
+					(size 1.27 1.27)
+				)
+			)
+		)
+		(property "Value" "Conn_02x08_Counter_Clockwise"
+			(at 238.76 129.54 0)
+			(effects
+				(font
+					(size 1.27 1.27)
+				)
+			)
+		)
+		(property "Footprint" "Connector_PinSocket_2.54mm:PinSocket_2x08_P2.54mm_Vertical"
+			(at 237.49 140.97 0)
+			(effects
+				(font
+					(size 1.27 1.27)
+				)
+				(hide yes)
+			)
+		)
+		(property "Datasheet" "~"
+			(at 237.49 140.97 0)
+			(effects
+				(font
+					(size 1.27 1.27)
+				)
+				(hide yes)
+			)
+		)
+		(property "Description" "Generic connector, double row, 02x08, counter clockwise pin numbering scheme (similar to DIP package numbering), script generated (kicad-library-utils/schlib/autogen/connector/)"
+			(at 237.49 140.97 0)
+			(effects
+				(font
+					(size 1.27 1.27)
+				)
+				(hide yes)
+			)
+		)
+		(pin "11"
+		)
+		(pin "4"
+		)
+		(pin "5"
+		)
+		(pin "6"
+		)
+		(pin "7"
+		)
+		(pin "1"
+		)
+		(pin "14"
+		)
+		(pin "10"
+		)
+		(pin "15"
+		)
+		(pin "16"
+		)
+		(pin "2"
+		)
+		(pin "3"
+		)
+		(pin "13"
+		)
+		(pin "8"
+		)
+		(pin "9"
+		)
+		(pin "12"
+		)
+		(instances
+			(project ""
+				(path "/880cd2ad-ee8a-45d0-bf92-2f93a861aac0/933c923e-9649-42a5-9bc4-db8878fb4adc"
+					(reference "J12")
+					(unit 1)
+				)

Commit message: branches
Parts:
- removed J10: Conn_02x06_Counter_Clockwise, Connector_PinHeader_2.54mm:PinHeader_2x06_P2.54mm_Vertical_SMD, symbol Connector_Generic:Conn_02x06_Counter_Clockwise
- added J13: Conn_02x06_Odd_Even, Connector_PinHeader_2.54mm:PinHeader_2x06_P2.54mm_Vertical_SMD, symbol Connector_Generic:Conn_02x06_Odd_Even
Connections:
- net GND: now also J11.6 (Pin_6), J13.11 (Pin_11), J13.12 (Pin_12)
- net PYRO_1: now also J13.1 (Pin_1)
- net PYRO_2: now also J13.3 (Pin_3)
- net PYRO_3: now also J13.5 (Pin_5)
- net PYRO_4: now also J13.7 (Pin_7)
- net +5V: now reaches J11.1 (Pin_1)
- net +5V: now also J13.10 (Pin_10)
- net TX_RFD900x: now reaches J11.2 (Pin_2)
- net RX_RFD900x: now reaches J11.3 (Pin_3)
- new net +3.3V: J13.9 (Pin_9)
- new net SCL_PM: J13.8 (Pin_8)
- new net SDA_PM: J13.6 (Pin_6)
- no-connect marks 0 -> 2
Other:
- note added: "can add hardware flow control here if desired"
- moved on the sheet: Q1
