File: SD.kicad_sch (KiCad schematic)
At the start: 1 part, among them J8 Micro_SD_Card

Commit message: routed🛣️
Parts:
- J8: footprint (none) -> Connector_Card:microSD_HC_Wuerth_693072010801
Changed lines of the file:
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@@
 			)
 		)
-		(property "Footprint" ""
+		(property "Footprint" "Connector_Card:microSD_HC_Wuerth_693072010801"
 			(at 179.07 91.44 0)
 			(effects

Commit message: branches
Other:
- note added: "Connect this Micro SD card to stm32. Use heirarchical labels"
Changed lines of the file:
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@@
+		)
+	)
+	(text "Connect this Micro SD card to stm32. Use heirarchical labels"
+		(exclude_from_sim no)
+		(at 106.934 58.928 0)
+		(effects
+			(font
+				(size 2.032 2.032)
+			)
 		)
 	)
