File: power.kicad_sch (KiCad schematic)
At the start: 0 parts

Commit message: power docs⚡️
Parts:
- added J1: Conn_01x02, Connector_AMASS:AMASS_XT30PW-M_1x02_P2.50mm_Horizontal, symbol Connector_Generic:Conn_01x02
Other:
- note added: "Need to implement two regs, 3.3v and 5v to run off of 2-3s lipo. Implement xt-30 connector for battery connection"
- note added: "Power"
Changed lines of the file:
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@@
 	(generator_version "8.0")
 	(paper "A4")
+	(text "Power"
+		(exclude_from_sim no)
+		(at 62.992 46.228 0)
+		(effects
+			(font
+				(size 2.032 2.032)
+			)
+		)
+	)
+	(text "Need to implement two regs, 3.3v and 5v to run off of 2-3s lipo.\nImplement xt-30 connector for battery connection"
+		(exclude_from_sim no)
+		(at 62.738 50.546 0)
+		(effects
+			(font
+				(size 1.27 1.27)
+			)
+		)
+	)
 	(symbol
 		(lib_id "power:+5V")
@@
 					(unit 1)
 				)
+			)
+		)
+	)
+	(symbol
+		(lib_id "Connector_Generic:Conn_01x02")
+		(at 90.17 87.63 180)
+		(unit 1)
+		(exclude_from_sim no)
+		(in_bom yes)
+		(on_board yes)
+		(dnp no)
+		(fields_autoplaced yes)
+		(property "Reference" "J1"
+			(at 90.17 78.74 0)
+			(effects
+				(font
+					(size 1.27 1.27)
+				)
+			)
+		)
+		(property "Value" "Conn_01x02"
+			(at 90.17 81.28 0)
+			(effects
+				(font
+					(size 1.27 1.27)
+				)
+			)
+		)
+		(property "Footprint" "Connector_AMASS:AMASS_XT30PW-M_1x02_P2.50mm_Horizontal"
+			(at 90.17 87.63 0)
+			(effects
+				(font
+					(size 1.27 1.27)
+				)
+				(hide yes)
+			)
+		)
+		(property "Datasheet" "~"
+			(at 90.17 87.63 0)
+			(effects
+				(font
+					(size 1.27 1.27)
+				)
+				(hide yes)
+			)
+		)
+		(property "Description" "Generic connector, single row, 01x02, script generated (kicad-library-utils/schlib/autogen/connector/)"
+			(at 90.17 87.63 0)
+			(effects
+				(font
+					(size 1.27 1.27)
+				)
+				(hide yes)
+			)
+		)
+		(pin "2"
+		)
+		(pin "1"
+		)
+		(instances
+			(project ""
+				(path "/880cd2ad-ee8a-45d0-bf92-2f93a861aac0/1713f0c2-87c4-4fc3-9379-51a871bad33e"
+					(reference "J1")
+					(unit 1)
+				)

Commit message: usb-c🔌
Parts:
- J1: footprint Connector_AMASS:AMASS_XT30PW-M_1x02_P2.50mm_Horizontal -> (none)
Other:
- note added: "From MCU USB port connected with diode"
- note added: "Need to implement two regs, 3.3v and 5v to run off of 2-3s lipo."
- note removed: "Need to implement two regs, 3.3v and 5v to run off of 2-3s lipo. Implement xt-30 connector for battery connection"
Changed lines of the file:
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@@
 		)
 	)
-	(text "Need to implement two regs, 3.3v and 5v to run off of 2-3s lipo.\nImplement xt-30 connector for battery connection"
+	(text "From MCU USB port connected with diode"
+		(exclude_from_sim no)
+		(at 166.878 109.22 0)
+		(effects
+			(font
+				(size 1.27 1.27)
+			)
+		)
+	)
+	(text "Need to implement two regs, 3.3v and 5v to run off of 2-3s lipo."
 		(exclude_from_sim no)
 		(at 62.738 50.546 0)
@@
 		)
 	)
+	(global_label "USB_VBUS"
+		(shape input)
+		(at 161.29 105.41 0)
+		(fields_autoplaced yes)
+		(effects
+			(font
+				(size 1.27 1.27)
+			)
+			(justify left)
+		)
+		(property "Intersheetrefs" "${INTERSHEET_REFS}"
+			(at 173.9514 105.41 0)
+			(effects
+				(font
+					(size 1.27 1.27)
+				)
+				(justify left)
+				(hide yes)
+			)
+		)
+	)
+	(symbol
+		(lib_id "Connector_Generic:Conn_01x02")
+		(at 105.41 87.63 180)
+		(unit 1)
+		(exclude_from_sim no)
+		(in_bom yes)
+		(on_board yes)
+		(dnp no)
+		(fields_autoplaced yes)
+		(property "Reference" "J1"
+			(at 105.41 78.74 0)
+			(effects
+				(font
+					(size 1.27 1.27)
+				)
+			)
+		)
+		(property "Value" "Conn_01x02"
+			(at 105.41 81.28 0)
+			(effects
+				(font
+					(size 1.27 1.27)
+				)
+			)
+		)
+		(property "Footprint" ""
+			(at 105.41 87.63 0)
+			(effects
+				(font
+					(size 1.27 1.27)
+				)
+				(hide yes)
+			)
+		)
+		(property "Datasheet" "~"
+			(at 105.41 87.63 0)
+			(effects
+				(font
+					(size 1.27 1.27)
+				)
+				(hide yes)
+			)
+		)
+		(property "Description" "Generic connector, single row, 01x02, script generated (kicad-library-utils/schlib/autogen/connector/)"
+			(at 105.41 87.63 0)
+			(effects
+				(font
+					(size 1.27 1.27)
+				)
+				(hide yes)
+			)
+		)
+		(pin "2"
+		)
+		(pin "1"
+		)
+		(instances
+			(project ""
+				(path "/880cd2ad-ee8a-45d0-bf92-2f93a861aac0/1713f0c2-87c4-4fc3-9379-51a871bad33e"
+					(reference "J1")
+					(unit 1)
+				)
+			)
+		)
+	)
 	(symbol
 		(lib_id "power:+5V")
@@
 					(unit 1)
 				)
-			)
-		)
-	)
-	(symbol
-		(lib_id "Connector_Generic:Conn_01x02")
-		(at 90.17 87.63 180)
-		(unit 1)
-		(exclude_from_sim no)
-		(in_bom yes)
-		(on_board yes)
-		(dnp no)
-		(fields_autoplaced yes)
-		(property "Reference" "J1"
-			(at 90.17 78.74 0)
-			(effects
-				(font
-					(size 1.27 1.27)
-				)
-			)
-		)
-		(property "Value" "Conn_01x02"
-			(at 90.17 81.28 0)
-			(effects
-				(font
-					(size 1.27 1.27)
-				)
-			)
-		)
-		(property "Footprint" "Connector_AMASS:AMASS_XT30PW-M_1x02_P2.50mm_Horizontal"
-			(at 90.17 87.63 0)
-			(effects
-				(font
-					(size 1.27 1.27)
-				)
-				(hide yes)
-			)
-		)
-		(property "Datasheet" "~"
-			(at 90.17 87.63 0)
-			(effects
-				(font
-					(size 1.27 1.27)
-				)
-				(hide yes)
-			)
-		)
-		(property "Description" "Generic connector, single row, 01x02, script generated (kicad-library-utils/schlib/autogen/connector/)"
-			(at 90.17 87.63 0)
-			(effects
-				(font
-					(size 1.27 1.27)
-				)
-				(hide yes)
-			)
-		)
-		(pin "2"
-		)
-		(pin "1"
-		)
-		(instances
-			(project ""
-				(path "/880cd2ad-ee8a-45d0-bf92-2f93a861aac0/1713f0c2-87c4-4fc3-9379-51a871bad33e"
-					(reference "J1")
-					(unit 1)
-				)

Commit message: mcu⚡️
Parts:
- removed J1: Conn_01x02, symbol Connector_Generic:Conn_01x02
- added C10: C, 4.7uF, symbol Device:C
- added C2, C3, C4, C5, C6, C7, C8, C9: C, 100nF, symbol Device:C
Connections:
- net +3.3V: now also C10.1, C2.1, C3.1, C4.1, C5.1, C6.1, C7.1, C8.1, C9.1
- new net GND: C10.2, C2.2, C3.2, C4.2, C5.2, C6.2, C7.2, C8.2, C9.2
Other:
- note added: "Decoupling for MCU"

Commit message: gps🌎
Other:
- note added: "Decoupling for MCU 8 x 100nF, 1 x 4.7uF"
- note removed: "Decoupling for MCU"
Changed lines of the file:
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@@
 		)
 	)
-	(text "Decoupling for MCU"
+	(text "Decoupling for MCU\n8 x 100nF, 1 x 4.7uF"
 		(exclude_from_sim no)
-		(at 229.362 73.66 0)
+		(at 226.568 74.168 0)
 		(effects
 			(font

Commit message: test
Parts:
- added C13: 10uF, Capacitor_SMD:C_0805_2012Metric, symbol Device:C
- added C14: 100nF, Capacitor_SMD:C_0402_1005Metric, symbol Device:C
- added C15, C16: 22uF, Capacitor_SMD:C_1206_3216Metric, symbol Device:C
- added L1: 4.7uH, Inductor_SMD:L_1008_2520Metric, symbol Device:L
- added U7: AP63203WU, Package_TO_SOT_SMD:TSOT-23-6, symbol Regulator_Switching:AP63203WU
- C10: value C -> 4.7uF; footprint 4.7uF -> Capacitor_SMD:C_0603_1608Metric
- C2, C3, C4, C5, C6, C7, C8, C9: value C -> 100nF; footprint 100nF -> Capacitor_SMD:C_0402_1005Metric
Connections:
- net +3.3V: now also C15.1, C16.1, L1.2, U7.1 (FB)
- net GND: now also C13.2, C15.2, C16.2, U7.4 (GND)
- new net: C14.1, L1.1, U7.5 (SW)
- new net: C14.2, U7.6 (BST)
- new net +BATT: C13.1, U7.2 (EN), U7.3 (IN)
Other:
- note added: "3.3v Switching Regulator"
- moved on the sheet: C10

Commit message: 5v⚡️
Parts:
- added C18: 0.1uF, Capacitor_SMD:C_0402_1005Metric, symbol Device:C
- added C19: 3.3nF, Capacitor_SMD:C_0402_1005Metric, symbol Device:C
- added C20: 22uF, Capacitor_SMD:C_1206_3216Metric, symbol Device:C
- added C21: 10uF, Capacitor_SMD:C_0805_2012Metric, symbol Device:C
- added L2: 2.2uH, Inductor_SMD:L_1008_2520Metric, symbol Device:L
- added R10: 100k, Resistor_SMD:R_0603_1608Metric, symbol Device:R
- added R11: 1M, Resistor_SMD:R_0603_1608Metric, symbol Device:R
- added R12: 200k, Resistor_SMD:R_0603_1608Metric, symbol Device:R
- added U9: TPS62130, Package_DFN_QFN:VQFN-16-1EP_3x3mm_P0.5mm_EP1.68x1.68mm_ThermalVias, symbol Regulator_Switching:TPS62130
Connections:
- net +5V: now also C20.1, L2.2, R10.1, R11.1, U9.14 (VOS), U9.7 (FSW)
- net +BATT: now also C18.2, C21.2, U9.10 (VIN), U9.11 (VIN), U9.12 (VIN), U9.13 (EN)
- net GND: now also C18.1, C19.2, C20.2, C21.1, R12.2, U9.15 (GND), U9.16 (GND), U9.17 (GND), U9.6 (GND), U9.8 (DEF)
- new net: R11.2, R12.1, U9.5 (FB)
- new net: C19.1, U9.9 (SS/TR)
- new net: L2.1, U9.1 (SW), U9.2 (SW), U9.3 (SW)
- new net: R10.2, U9.4 (PG)
Other:
- note added: "5v Switching Regulator"
- note added: "R11 = R12((Vout/0.8V) - 1)"

Commit message: computer
Other:
- note added: "Global Current Sensing"
Changed lines of the file:
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@@
+	)
+	(rectangle
+		(start 128.27 100.33)
+		(end 218.44 137.16)
+		(stroke
+			(width 0)
+			(type default)
+		)
+		(fill
+			(type none)
+		)
 	)
 	(rectangle
@@
 		(effects
 			(font
+				(size 2.032 2.032)
+			)
+		)
+	)
+	(text "Global Current Sensing\n"
+		(exclude_from_sim no)
+		(at 147.32 97.282 0)
+		(effects
+			(font

Commit message: branches
Parts:
- removed C10: 4.7uF, Capacitor_SMD:C_0603_1608Metric, symbol Device:C
- removed C2, C3, C4, C5, C6, C7, C8, C9: 100nF, Capacitor_SMD:C_0402_1005Metric, symbol Device:C
- removed U9: TPS62130, Package_DFN_QFN:VQFN-16-1EP_3x3mm_P0.5mm_EP1.68x1.68mm_ThermalVias, symbol Regulator_Switching:TPS62130
- added C22: 2.2uF, Capacitor_SMD:C_0603_1608Metric, symbol Device:C
- added C23: 100nF, Capacitor_SMD:C_0402_1005Metric, symbol Device:C
- added C24: 470pF, Capacitor_SMD:C_0402_1005Metric, symbol Device:C
- added C25, C26, C27, C28: 22uF, Capacitor_SMD:C_1206_3216Metric, symbol Device:C
- added PS1: TPS513885VABR, TPS513885VABR:CONV_TPS513885VABR, symbol TPS513885VABR:TPS513885VABR
- added R17: R, symbol Device:R
- C18: value 0.1uF -> 100nF
- C19: value 3.3nF -> 22uF; footprint Capacitor_SMD:C_0402_1005Metric -> Capacitor_SMD:C_1206_3216Metric
- C21: value 10uF -> 22uF; footprint Capacitor_SMD:C_0805_2012Metric -> Capacitor_SMD:C_1206_3216Metric
- L2: value 2.2uH -> 1.5uH
- R11: value 1M -> 0; footprint Resistor_SMD:R_0603_1608Metric -> (none)
- R12: value 200k -> 1k; footprint Resistor_SMD:R_0603_1608Metric -> Resistor_SMD:R_0402_1005Metric
Connections:
- net +3.3V: now also PS1.5 (MODE), PS1.6 (EN)
- net +5V: now also C25.1, C26.1, C27.1, C28.1, R17.1; no longer C20.1, R10.1, R11.1
- net +BATT: now also C18.1, C19.1, C20.1, C21.1, PS1.1 (VIN); no longer C18.2, C21.2
- net GND: now also C18.2, C21.2, C22.1, PS1.11 (PGND), PS1.3 (PGND); no longer C18.1, C21.1, R12.2
- net at R11.2: now also PS1.13 (VBST); no longer R12.1
- net at L2.1: now also C23.2, PS1.12 (SW), PS1.2 (SW)
- net at R10.2: now also C22.2, PS1.10 (VCC)
- new net: PS1.4 (PG), R10.1
- new net: PS1.7 (FB), R12.2
- new net: C24.2, R12.1
- new net: C23.1, R11.1
- new net FB: C24.1, C25.2, C26.2, C27.2, C28.2, PS1.8 (VOUT), R17.2
- no-connect marks 0 -> 1
Other:
- note added: "TODO: ensure all parts here are rated for voltage/amperage"
- note removed: "Decoupling for MCU 8 x 100nF, 1 x 4.7uF"
- note removed: "R11 = R12((Vout/0.8V) - 1)"
- moved on the sheet: C13, C14, C15, C16, L1, U7
