File: untitled.kicad_sch (KiCad schematic)
At the start: 1 part, among them U10 SP3485EN

Commit message: branches
Parts:
- added J4: Conn_01x02, Connector_JST:JST_PH_S2B-PH-K_1x02_P2.00mm_Horizontal, symbol Connector_Generic:Conn_01x02
Connections:
- net RX_RS485: now reaches U10.1 (RO)
- net DIR_RS485: now reaches U10.2 (~{RE})
- net DIR_RS485: now also U10.3 (DE)
- net TX_RS485: now reaches U10.4 (DI)
- net GND: now reaches U10.5 (GND)
- net at U10.6 (A): now also J4.1 (Pin_1)
- net at U10.7 (B): now also J4.2 (Pin_2)
- net +3.3V: now reaches U10.8 (VCC)
