File: Compute-Comms/power.kicad_sch (KiCad schematic)
At the start: 43 parts, among them J1 Conn_01x02, J5 Conn_01x02, J6 Conn_01x02, J7 Conn_01x02, Q1 SSM3J328R, Q2 SSM3J328R, Q3 L2N7002SLLT1G, Q4 L2N7002SLLT1G, Q5 SSM3J328R, Q6 SSM3J328R, Q7 L2N7002SLLT1G, Q8 L2N7002SLLT1G, U7 AP63203WU

Commit message: separate⚮
Parts:
- removed C13: 10uF, Capacitor_SMD:C_0805_2012Metric, symbol Device:C
- removed C14, C18, C23: 100nF, Capacitor_SMD:C_0402_1005Metric, symbol Device:C
- removed C15, C16, C19, C20, C21, C25, C26, C27, C28: 22uF, Capacitor_SMD:C_1206_3216Metric, symbol Device:C
- removed C22: 2.2uF, Capacitor_SMD:C_0603_1608Metric, symbol Device:C
- removed C24: 470pF, Capacitor_SMD:C_0402_1005Metric, symbol Device:C
- removed J1, J5, J6, J7: Conn_01x02, symbol Connector_Generic:Conn_01x02
- removed L1: 4.7uH, Inductor_SMD:L_1008_2520Metric, symbol Device:L
- removed L2: 1.5uH, Inductor_SMD:L_1008_2520Metric, symbol Device:L
- removed PS1: TPS513885VABR, TPS513885VABR:CONV_TPS513885VABR, symbol TPS513885VABR:TPS513885VABR
- removed Q1, Q2, Q5, Q6: SSM3J328R, SSM3J328R:SOT95P240X88-3N, symbol Simulation_SPICE:PMOS
- removed Q3, Q4, Q7, Q8: L2N7002SLLT1G, Package_TO_SOT_SMD:SOT-23, symbol Simulation_SPICE:NMOS
- removed R10, R13, R14, R15, R16, R4, R5, R8, R9: 100k, Resistor_SMD:R_0603_1608Metric, symbol Device:R
- removed R11: 0, symbol Device:R
- removed R12: 1k, Resistor_SMD:R_0402_1005Metric, symbol Device:R
- removed R17: R, symbol Device:R
- removed U7: AP63203WU, Package_TO_SOT_SMD:TSOT-23-6, symbol Regulator_Switching:AP63203WU
Connections:
- no-connect marks 1 -> 0
Other:
- note removed: "3.3v Switching Regulator"
- note removed: "5v Switching Regulator"
- note removed: "Found this pmos by digikey, 20v, in stock, pmos, scrolling for high amperage"
- note removed: "From MCU USB port connected with diode"
- note removed: "Global Current Sensing"
- note removed: "Need to implement two regs, 3.3v and 5v to run off of 2-3s lipo."
- note removed: "Power"
- note removed: "Pyro Channels"
- note removed: "SSM3J328R PMOS"
- note removed: "TODO: ensure all parts here are rated for voltage/amperage"
- note removed: "Use this for VBAT level Pyro"
