File: Compute-Comms/LoRa.kicad_sch (KiCad schematic)
At the start: 2 parts, among them J9 Conn_01x01, U11 Ai-Thinker-Ra-01

Commit message: FERBBBB🟣
Parts:
- J9: footprint TestPoint:TestPoint_THTPad_D3.0mm_Drill1.5mm -> TestPoint:TestPoint_Keystone_5015_Micro-Minature
Changed lines of the file:
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@@
 			)
 		)
-		(property "Footprint" "TestPoint:TestPoint_THTPad_D3.0mm_Drill1.5mm"
+		(property "Footprint" "TestPoint:TestPoint_Keystone_5015_Micro-Minature"
 			(at 171.45 82.55 0)
 			(effects
