File: Compute-Comms/NDXPCOMPUTER.kicad_sch (KiCad schematic)
At the start: 0 parts

Commit message: separate⚮
Other:
- removed sheet Power
Changed lines of the file:
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@@
-	)
-	(sheet
-		(at 71.12 55.88)
-		(size 25.4 22.86)
-		(stroke
-			(width 0.1524)
-			(type solid)
-		)
-		(fill
-			(color 0 0 0 0.0000)
-		)
-		(property "Sheetname" "Power"
-			(at 80.264 68.072 0)
-			(effects
-				(font
-					(size 1.27 1.27)
-				)
-				(justify left bottom)
-			)
-		)
-		(property "Sheetfile" "power.kicad_sch"
-			(at 71.12 79.3246 0)
-			(effects
-				(font
-					(size 1.27 1.27)
-				)
-				(justify left top)
-			)
-		)
-		(instances
-			(project "NDXPCOMPUTER"
-				(path "/880cd2ad-ee8a-45d0-bf92-2f93a861aac0"
-					(page "7")
-				)
-			)
-		)
 	)
 	(sheet
@@
 	)
 	(sheet
-		(at 99.06 35.56)
+		(at 88.9 52.07)
 		(size 21.59 16.51)
 		(stroke
@@
 		)
 		(property "Sheetname" "SD"
-			(at 108.458 44.45 0)
+			(at 98.298 60.96 0)
 			(effects
 				(font
@@
 		)
 		(property "Sheetfile" "SD.kicad_sch"
-			(at 98.806 52.578 0)
+			(at 88.646 69.088 0)
 			(effects
 				(font

Commit message: sd♠️
Changed lines of the file:
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@@
 	(wire
 		(pts
-			(xy 102.87 99.06) (xy 121.92 99.06)
+			(xy 102.87 109.22) (xy 121.92 109.22)
 		)
 		(stroke
@@
 	(wire
 		(pts
-			(xy 102.87 93.98) (xy 121.92 93.98)
+			(xy 102.87 104.14) (xy 121.92 104.14)
 		)
 		(stroke
@@
 	(wire
 		(pts
-			(xy 102.87 91.44) (xy 121.92 91.44)
+			(xy 102.87 101.6) (xy 121.92 101.6)
 		)
 		(stroke
@@
 	(wire
 		(pts
-			(xy 102.87 96.52) (xy 121.92 96.52)
+			(xy 102.87 106.68) (xy 121.92 106.68)
 		)
 		(stroke
@@
 		)
 		(pin "PYRO_1" input
-			(at 102.87 91.44 0)
+			(at 102.87 101.6 0)
 			(effects
 				(font
@@
 		)
 		(pin "PYRO_3" input
-			(at 102.87 96.52 0)
+			(at 102.87 106.68 0)
 			(effects
 				(font
@@
 		)
 		(pin "PYRO_2" input
-			(at 102.87 93.98 0)
+			(at 102.87 104.14 0)
 			(effects
 				(font
@@
 		)
 		(pin "PYRO_4" input
-			(at 102.87 99.06 0)
+			(at 102.87 109.22 0)
 			(effects
 				(font
@@
 		)
 		(pin "PYRO_3" input
-			(at 121.92 96.52 180)
+			(at 121.92 106.68 180)
 			(effects
 				(font
@@
 		)
 		(pin "PYRO_1" input
-			(at 121.92 91.44 180)
+			(at 121.92 101.6 180)
 			(effects
 				(font
@@
 		)
 		(pin "PYRO_2" input
-			(at 121.92 93.98 180)
+			(at 121.92 104.14 180)
 			(effects
 				(font
@@
 		)
 		(pin "PYRO_4" input
-			(at 121.92 99.06 180)
-			(effects
-				(font
+			(at 121.92 109.22 180)
+			(effects
+				(font

Commit message: 🔌
Other:
- note added: "TODO"
- note added: "make sure all i2c have pullup resistors Connect SD Card Rework GPS for UART Add Servo PWM pads in Peripherals Wire Breakout Pads"
Changed lines of the file:
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@@
+		)
+	)
+	(text "make sure all i2c have pullup resistors\nConnect SD Card\nRework GPS for UART\nAdd Servo PWM pads in Peripherals\nWire Breakout Pads\n"
+		(exclude_from_sim no)
+		(at 87.376 32.766 0)
+		(effects
+			(font
+				(size 1.27 1.27)
+			)
+		)
+	)
+	(text "TODO"
+		(exclude_from_sim no)
+		(at 87.63 25.4 0)
+		(effects
+			(font
+				(size 2.54 2.54)
+			)
 		)
 	)

Commit message: test
Other:
- note added: "make sure all i2c have pullup resistors Connect SD Card Rework GPS for UART Add Servo PWM pads in Peripherals Wire Breakout Pads Add cool leds"
- note removed: "make sure all i2c have pullup resistors Connect SD Card Rework GPS for UART Add Servo PWM pads in Peripherals Wire Breakout Pads"
Changed lines of the file:
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@@
 		)
 	)
-	(text "make sure all i2c have pullup resistors\nConnect SD Card\nRework GPS for UART\nAdd Servo PWM pads in Peripherals\nWire Breakout Pads\n"
+	(text "make sure all i2c have pullup resistors\nConnect SD Card\nRework GPS for UART\nAdd Servo PWM pads in Peripherals\nWire Breakout Pads\nAdd cool leds\n"
 		(exclude_from_sim no)
-		(at 87.376 32.766 0)
+		(at 87.376 33.274 0)
 		(effects
 			(font
