File: Compute-Comms/NEO-M9N.kicad_sch (KiCad schematic)
At the start: 3 parts, among them J3 Conn_Coaxial, U5 NEO-M9N

Commit message: Diff🍐
Changed lines of the file:
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@@
 (kicad_sch
-	(version 20231120)
+	(version 20250114)
 	(generator "eeschema")
-	(generator_version "8.0")
+	(generator_version "9.0")
 	(paper "A4")
+	(text "Low for spi\n"
+		(exclude_from_sim no)
+		(at 110.998 120.142 0)
+		(effects
+			(font
+				(size 1.27 1.27)
+			)
+		)
+	)
 	(junction
 		(at 133.35 78.74)
@@
 		)
 	)
-	(text "Low for spi\n"
-		(exclude_from_sim no)
-		(at 110.998 120.142 0)
-		(effects
-			(font
-				(size 1.27 1.27)
-			)
-		)
-	)
 	(hierarchical_label "DI_GPS"
 		(shape input)
 		(at 120.65 96.52 180)
-		(fields_autoplaced yes)
 		(effects
 			(font
@@
 		(shape input)
 		(at 120.65 104.14 180)
-		(fields_autoplaced yes)
 		(effects
 			(font
@@
 		(shape input)
 		(at 120.65 93.98 180)
-		(fields_autoplaced yes)
 		(effects
 			(font
@@
 		(shape input)
 		(at 120.65 101.6 180)
-		(fields_autoplaced yes)
 		(effects
 			(font
