File: Compute-Comms/Peripherals.kicad_sch (KiCad schematic)
At the start: 27 parts, among them J1 Conn_01x02, J11 Conn_01x06, J12 Conn_02x08_Counter_Clockwise, J13 Conn_02x06_Odd_Even, J5 Conn_01x02, J6 Conn_01x02, J7 Conn_01x02, Q1 SSM3J328R, Q2 L2N7002SLLT1G, Q3 SSM3J328R, Q4 L2N7002SLLT1G, Q5 SSM3J328R, Q6 L2N7002SLLT1G, Q7 SSM3J328R, Q8 L2N7002SLLT1G

Commit message: refactor🧮
Parts:
- removed J1, J5, J6, J7: Conn_01x02, symbol Connector_Generic:Conn_01x02
- removed Q1, Q3, Q5, Q7: SSM3J328R, SSM3J328R:SOT95P240X88-3N, symbol Simulation_SPICE:PMOS
- removed Q2, Q4, Q6, Q8: L2N7002SLLT1G, Package_TO_SOT_SMD:SOT-23, symbol Simulation_SPICE:NMOS
- removed R13, R14, R15, R16, R4, R5, R8, R9: 100k, Resistor_SMD:R_0603_1608Metric, symbol Device:R
Other:
- note removed: "Found this pmos by digikey, 20v, in stock, pmos, scrolling for high amperage"
- note removed: "Pyro Channels"
- note removed: "SSM3J328R PMOS"
- note removed: "Use this for VBAT level Pyro"

Commit message: separate⚮
Other:
- note added: "Breakout Spare 3 UARTS, 1x I2C, 1xSPI, 5v, 3v, 2x GND"
- note removed: "Breakout Spare UARTS, 1x I2C, 1xSPI, 5v, 3v,"
- moved on the sheet: H1, H2, H3, H4, J11, J12, J13

Commit message: sd♠️
Changed lines of the file:
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@@
+		(color 0 0 0 0)
+	)
+	(junction
+		(at 99.06 85.09)
+		(diameter 0)
 		(color 0 0 0 0)
 	)
@@
 					(unit 1)
 				)
+			)
+		)
+	)
+	(symbol
+		(lib_id "power:PWR_FLAG")
+		(at 99.06 85.09 180)
+		(unit 1)
+		(exclude_from_sim no)
+		(in_bom yes)
+		(on_board yes)
+		(dnp no)
+		(fields_autoplaced yes)
+		(property "Reference" "#FLG02"
+			(at 99.06 86.995 0)
+			(effects
+				(font
+					(size 1.27 1.27)
+				)
+				(hide yes)
+			)
+		)
+		(property "Value" "PWR_FLAG"
+			(at 99.06 90.17 0)
+			(effects
+				(font
+					(size 1.27 1.27)
+				)
+			)
+		)
+		(property "Footprint" ""
+			(at 99.06 85.09 0)
+			(effects
+				(font
+					(size 1.27 1.27)
+				)
+				(hide yes)
+			)
+		)
+		(property "Datasheet" "~"
+			(at 99.06 85.09 0)
+			(effects
+				(font
+					(size 1.27 1.27)
+				)
+				(hide yes)
+			)
+		)
+		(property "Description" "Special symbol for telling ERC where power comes from"
+			(at 99.06 85.09 0)
+			(effects
+				(font
+					(size 1.27 1.27)
+				)
+				(hide yes)
+			)
+		)
+		(pin "1"
+		)
+		(instances
+			(project "NDXPCOMPUTER"
+				(path "/880cd2ad-ee8a-45d0-bf92-2f93a861aac0/933c923e-9649-42a5-9bc4-db8878fb4adc"
+					(reference "#FLG02")
+					(unit 1)
+				)
