File: Compute-Comms/STM32H7.kicad_sch (KiCad schematic)
At the start: 23 parts, among them J2 USB_C_Receptacle_USB2.0_16P, SW1 SW_Push, SW2 SW_Push, U1 STM32H723VGTx

Commit message: separate⚮
Connections:
- net USB_VBUS renamed +5V
Other:
- note added: "From MCU USB port connected with diode"

Commit message: test
Connections:
- net +5V renamed +BATT

Commit message: Diff🍐
Parts:
- R6, R7: footprint Resistor_SMD:R_0603_1608Metric -> Resistor_SMD:R_0201_0603Metric
Changed lines of the file:
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@@
 (kicad_sch
-	(version 20231120)
+	(version 20250114)
 	(generator "eeschema")
-	(generator_version "8.0")
+	(generator_version "9.0")
 	(paper "A4")
