File: Compute-Comms/untitled.kicad_sch (KiCad schematic)
At the start: 2 parts, among them J4 Conn_01x02, U10 SP3485EN

Commit message: FERBBBB🟣
Parts:
- J4: footprint Connector_JST:JST_PH_S2B-PH-K_1x02_P2.00mm_Horizontal -> SM02B-GHS:CONN_SM02B-GHS_JST
Changed lines of the file:
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@@
 			)
 		)
-		(property "Footprint" "Connector_JST:JST_PH_S2B-PH-K_1x02_P2.00mm_Horizontal"
+		(property "Footprint" "SM02B-GHS:CONN_SM02B-GHS_JST"
 			(at 171.45 88.9 0)
 			(effects
