File: Compute-Comms/NDXPCOMPUTER.kicad_pcb (KiCad board)
At the start: 2 copper layers, 31.4 x 55.6 mm, 84 parts, among them IC1 IIS2MDCTR, J11 Conn_01x06, J12 Conn_02x08_Counter_Clockwise, J13 Conn_02x06_Odd_Even, J2 USB_C_Receptacle_USB2.0_16P, J3 Conn_Coaxial, J4 Conn_01x02, J8 Micro_SD_Card, J9 Conn_01x01, Q1 SSM3J328R, Q2 L2N7002SLLT1G, Q3 SSM3J328R, Q4 L2N7002SLLT1G, Q5 SSM3J328R, Q6 L2N7002SLLT1G, Q7 SSM3J328R, Q8 L2N7002SLLT1G, SW1 SW_Push, SW2 SW_Push, U1 STM32H723VGTx, U10 SP3485EN, U11 Ai-Thinker-Ra-01, U2 BMI088, U3 LSM6DSM, U4 BMP581, U5 NEO-M9N, U7 AP63203WU

Commit message: sd♠️
Parts:
- removed C13: 10uF, Capacitor_SMD:C_0805_2012Metric
- removed C14, C18, C23: 100nF, Capacitor_SMD:C_0402_1005Metric
- removed C15, C16, C19, C20, C21, C25, C26, C27, C28: 22uF, Capacitor_SMD:C_1206_3216Metric
- removed C22: 2.2uF, Capacitor_SMD:C_0603_1608Metric
- removed C24: 470pF, Capacitor_SMD:C_0402_1005Metric
- removed L1: 4.7uH, Inductor_SMD:L_1008_2520Metric
- removed L2: 1.5uH, Inductor_SMD:L_1008_2520Metric
- removed PS1: TPS513885VABR, TPS513885VABR:CONV_TPS513885VABR
- removed Q1, Q3, Q5, Q7: SSM3J328R, SSM3J328R:SOT95P240X88-3N
- removed Q2, Q4, Q6, Q8: L2N7002SLLT1G, Package_TO_SOT_SMD:SOT-23
- removed R10, R13, R14, R15, R16, R4, R5, R8, R9: 100k, Resistor_SMD:R_0603_1608Metric
- removed R12: 1k, Resistor_SMD:R_0402_1005Metric
- removed U7: AP63203WU, Package_TO_SOT_SMD:TSOT-23-6
- J8: moved to B.Cu
- moved J8 54.0 mm to (147.8, 109.9), turned to 90 degrees
- moved J9 34.7 mm to (107.6, 112.9)
- moved G*** 24.5 mm to (152.6, 106.3)
- moved C1 23.4 mm to (93.0, 112.0)
- moved C11 23.4 mm to (89.5, 106.1)
- moved C2 23.4 mm to (93.0, 114.0)
- moved C3 23.4 mm to (93.0, 116.0)
- moved C4 23.4 mm to (95.9, 112.0)
- moved C5 23.4 mm to (95.9, 114.0)
- moved C6 23.4 mm to (95.9, 116.0)
- moved C7 23.4 mm to (98.7, 112.0)
- moved C8 23.4 mm to (98.7, 114.0)
- moved C9 23.4 mm to (98.7, 116.0)
- moved R2 23.4 mm to (101.6, 114.0)
- moved R3 23.4 mm to (101.6, 116.0)
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Connections:
- net USB_VBUS renamed +5V
Other:
- board size 31.4 x 55.6 mm -> 31.5 x 55.5 mm

Commit message: FERBBBB🟣
Parts:
- removed J8: Micro_SD_Card, Connector_Card:microSD_HC_Wuerth_693072010801
- added MICRO_SD1: TF-01A, TF-01A:TF-01A, B.Cu at (147.3, 108.1)
- J4: footprint Connector_JST:JST_PH_S2B-PH-K_1x02_P2.00mm_Horizontal -> SM02B-GHS:CONN_SM02B-GHS_JST; moved to B.Cu
- J9: footprint TestPoint:TestPoint_THTPad_D3.0mm_Drill1.5mm -> TestPoint:TestPoint_Keystone_5015_Micro-Minature; moved to B.Cu
- R6, R7: moved to B.Cu
- moved C11 60.4 mm to (149.2, 115.6)
- moved C12 59.4 mm to (148.4, 100.4)
- moved JP1 54.1 mm to (152.8, 114.1), turned to 180 degrees
- moved SW1 53.9 mm to (147.8, 96.9), turned to 90 degrees
- moved R6 49.1 mm to (138.3, 105.3), turned to -90 degrees
- moved R7 49.0 mm to (138.3, 108.3), turned to 90 degrees
- moved J9 45.0 mm to (132.0, 75.1), turned to 90 degrees
- moved C1 41.9 mm to (133.2, 100.2), turned to -90 degrees
- moved R2 41.2 mm to (142.6, 117.8)
- moved C3 39.8 mm to (131.0, 104.2), turned to 90 degrees
- moved SW2 39.2 mm to (131.8, 96.8), turned to 90 degrees
- moved C10 39.2 mm to (128.7, 101.7), turned to 90 degrees
- moved C2 38.8 mm to (131.0, 106.1), turned to -90 degrees
- moved R1 37.1 mm to (138.3, 117.8)
- moved J4 36.5 mm to (128.0, 117.5), turned to 90 degrees
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Other:
- board text added: "RS-485"
- board text added: "Telemetry"

Commit message: baller🏀
Parts:
- added G***: LOGO, Images:Untitled, B.Cu at (135.0, 111.3)
- moved R2 1.79 mm to (140.8, 117.8)
- turned C11 to 180 degrees
- turned U4 to 90 degrees
Routing:
- net /LoRa/CS_LORA: track 0.00 -> 25.3 mm, vias 0 -> 1
- net /BMP581/SCK_BARO: track 0.00 -> 20.7 mm, vias 0 -> 1
- net /LoRa/RST_LORA: track 0.00 -> 19.4 mm, vias 0 -> 1
- net /BMP581/SDO_BARO: track 0.00 -> 13.6 mm
- net /BMP581/SDI_BARO: track 0.00 -> 12.5 mm
- net /LSM6DSM/SCL_IMU_LOW: track 0.00 -> 10.3 mm, vias 0 -> 2
- net /LSM6DSM/CS_IMU_LOW: track 0.00 -> 10.1 mm
- net Net-(U1-BOOT0): track 0.00 -> 9.95 mm
- net /LSM6DSM/SDO_IMU_LOW: track 0.00 -> 7.86 mm, vias 0 -> 2
- net /BMP581/CS_BARO: track 0.00 -> 7.17 mm
- net /BMI088/CS_GYRO: track 0.00 -> 6.50 mm
- net /Peripherals/PYRO_4: track 0.00 -> 5.04 mm, vias 0 -> 1
- net Net-(C11-Pad2): track 0.00 -> 4.24 mm
- net /Peripherals/PYRO_3: track 0.00 -> 4.05 mm, vias 0 -> 1
- net /Peripherals/PYRO_1: track 0.00 -> 3.97 mm, vias 0 -> 1
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- added copper zone on F.Cu, net +3.3V
- added copper zone on B.Cu, net GND
Other:
- board text added: "Boot"
- board text added: "Reset"

Commit message: test
Parts:
- moved J3 0.43 mm to (140.3, 75.8)
Connections:
- D1 pad 1: +5V -> +BATT
Routing:
- net Net-(J3-In): track 0.00 -> 21.5 mm
- net GND: vias 0 -> 39
- added copper zone on F.Cu, net GND
- removed copper zone on F.Cu, net +3.3V
Other:
- copper layers 2 -> 4

Commit message: Diff🍐
Parts:
- R6, R7: footprint Resistor_SMD:R_0603_1608Metric -> Resistor_SMD:R_0201_0603Metric; moved to F.Cu
- moved J9 16.5 mm to (148.5, 75.0)
- moved R7 11.9 mm to (149.4, 104.1)
- moved R6 11.1 mm to (149.4, 105.3)
- turned JP1 to 0 degrees
Routing:
- net D-: track 0.00 -> 35.0 mm, vias 0 -> 2
- net D+: track 0.00 -> 35.0 mm, vias 0 -> 2
- added copper zone on In2.Cu, net +3.3V
- added copper zone on In1.Cu, net GND

Commit message: some⛓️‍💥
Parts:
- added D2: LED, LED_SMD:LED_01005_0402Metric, B.Cu at (136.4, 103.6)
- added D3: LED, LED_SMD:LED_01005_0402Metric, B.Cu at (134.8, 103.6)
