File: Power-Pyro/NDXPPOWER.kicad_sch (KiCad schematic)
At the start: 47 parts, among them J1 Conn_01x02, J2 Conn_01x02, J3 Conn_01x02, J5 Conn_01x02, Q1 SSM3J328R, Q2 SSM3J328R, Q3 L2N7002SLLT1G, Q4 L2N7002SLLT1G, Q5 SSM3J328R, Q6 SSM3J328R, Q7 L2N7002SLLT1G, Q8 L2N7002SLLT1G, U1 AP63203WU

Commit message: hi
Other:
- added sheet Current Sense (current_sense.kicad_sch)
Changed lines of the file:
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@@
 (kicad_sch
-	(version 20231120)
+	(version 20250114)
 	(generator "eeschema")
-	(generator_version "8.0")
+	(generator_version "9.0")
 	(paper "A4")
+	(rectangle
+		(start 21.59 127)
+		(end 167.64 193.04)
+		(stroke
+			(width 0)
+			(type default)
+		)
+		(fill
+			(type none)
+		)
+	)
+	(rectangle
+		(start 21.59 81.28)
+		(end 111.76 118.11)
+		(stroke
+			(width 0)
+			(type default)
+		)
+		(fill
+			(type none)
+		)
+	)
+	(rectangle
+		(start 167.64 15.24)
+		(end 273.05 118.11)
+		(stroke
+			(width 0)
+			(type default)
+		)
+		(fill
+			(type none)
+		)
+	)
+	(rectangle
+		(start 121.92 81.28)
+		(end 162.56 118.11)
+		(stroke
+			(width 0)
+			(type default)
+		)
+		(fill
+			(type none)
+		)
+	)
+	(text "SSM3J328R PMOS\n"
+		(exclude_from_sim no)
+		(at 181.864 73.152 0)
+		(effects
+			(font
+				(size 1.27 1.27)
+			)
+		)
+	)
+	(text "Found this pmos by digikey, 20v, in stock, \npmos, scrolling for high amperage"
+		(exclude_from_sim no)
+		(at 180.848 17.526 0)
+		(effects
+			(font
+				(size 0.762 0.762)
+			)
+		)
+	)
+	(text "TODO: ensure all parts here are rated for voltage/amperage"
+		(exclude_from_sim no)
+		(at 52.578 83.058 0)
+		(effects
+			(font
+				(size 1.27 1.27)
+			)
+		)
+	)
+	(text "SSM3J328R PMOS\n"
+		(exclude_from_sim no)
+		(at 226.314 74.422 0)
+		(effects
+			(font
+				(size 1.27 1.27)
+			)
+		)
+	)
+	(text "Power"
+		(exclude_from_sim no)
+		(at 56.642 43.688 0)
+		(effects
+			(font
+				(size 2.032 2.032)
+			)
+		)
+	)
+	(text "SSM3J328R PMOS\n"
+		(exclude_from_sim no)
+		(at 225.044 26.162 0)
+		(effects
+			(font
+				(size 1.27 1.27)
+			)
+		)
+	)
+	(text "From MCU USB port connected with diode"
+		(exclude_from_sim no)
+		(at 98.298 68.58 0)
+		(effects
+			(font
+				(size 1.27 1.27)
+			)
+		)
+	)
+	(text "Use this for VBAT level Pyro"
+		(exclude_from_sim no)
+		(at 214.63 17.272 0)
+		(effects
+			(font
+				(size 1.27 1.27)
+			)
+		)
+	)
+	(text "Pyro Channels"
+		(exclude_from_sim no)
+		(at 182.626 14.224 0)
+		(effects
+			(font
+				(size 1.27 1.27)
+			)
+		)
+	)
+	(text "SSM3J328R PMOS\n"
+		(exclude_from_sim no)
+		(at 181.864 24.892 0)
+		(effects
+			(font
+				(size 1.27 1.27)
+			)
+		)
+	)
+	(text "5v Switching Regulator"
+		(exclude_from_sim no)
+		(at 40.386 124.206 0)
+		(effects
+			(font
+				(size 2.032 2.032)
+			)
+		)
+	)
+	(text "Global Current Sensing\n"
+		(exclude_from_sim no)
+		(at 140.97 78.232 0)
+		(effects
+			(font
+				(size 2.032 2.032)
+			)
+		)
+	)
+	(text "Need to implement two regs, 3.3v and 5v to run off of 2-3s lipo."
+		(exclude_from_sim no)
+		(at 56.388 48.006 0)
+		(effects
+			(font
+				(size 1.27 1.27)
+			)
+		)
+	)
+	(text "TODO: ensure all parts here are rated for voltage/amperage"
+		(exclude_from_sim no)
+		(at 96.012 130.048 0)
+		(effects
+			(font
+				(size 1.27 1.27)
+			)
+		)
+	)
+	(text "3.3v Switching Regulator\n"
+		(exclude_from_sim no)
+		(at 40.64 78.232 0)
+		(effects
+			(font
+				(size 2.032 2.032)
+			)
+		)
+	)
 	(junction
 		(at 87.63 88.9)
@@
 		)
 	)
-	(rectangle
-		(start 21.59 127)
-		(end 167.64 193.04)
-		(stroke
-			(width 0)
-			(type default)
-		)
-		(fill
-			(type none)
-		)
-	)
-	(rectangle
-		(start 21.59 81.28)
-		(end 111.76 118.11)
-		(stroke
-			(width 0)
-			(type default)
-		)
-		(fill
-			(type none)
-		)
-	)
-	(rectangle
-		(start 167.64 15.24)
-		(end 273.05 118.11)
-		(stroke
-			(width 0)
-			(type default)
-		)
-		(fill
-			(type none)
-		)
-	)
-	(rectangle
-		(start 121.92 81.28)
-		(end 162.56 118.11)
-		(stroke
-			(width 0)
-			(type default)
-		)
-		(fill
-			(type none)
-		)
-	)
-	(text "SSM3J328R PMOS\n"
-		(exclude_from_sim no)
-		(at 181.864 73.152 0)
-		(effects
-			(font
-				(size 1.27 1.27)
-			)
-		)
-	)
-	(text "Found this pmos by digikey, 20v, in stock, \npmos, scrolling for high amperage"
-		(exclude_from_sim no)
-		(at 180.848 17.526 0)
-		(effects
-			(font
-				(size 0.762 0.762)
-			)
-		)
-	)
-	(text "TODO: ensure all parts here are rated for voltage/amperage"
-		(exclude_from_sim no)
-		(at 52.578 83.058 0)
-		(effects
-			(font
-				(size 1.27 1.27)
-			)
-		)
-	)
-	(text "SSM3J328R PMOS\n"
-		(exclude_from_sim no)
-		(at 226.314 74.422 0)
-		(effects
-			(font
-				(size 1.27 1.27)
-			)
-		)
-	)
-	(text "Power"
-		(exclude_from_sim no)
-		(at 56.642 43.688 0)
-		(effects
-			(font
-				(size 2.032 2.032)
-			)
-		)
-	)
-	(text "SSM3J328R PMOS\n"
-		(exclude_from_sim no)
-		(at 225.044 26.162 0)
-		(effects
-			(font
-				(size 1.27 1.27)
-			)
-		)
-	)
-	(text "From MCU USB port connected with diode"
-		(exclude_from_sim no)
-		(at 98.298 68.58 0)
-		(effects
-			(font
-				(size 1.27 1.27)
-			)
-		)
-	)
-	(text "Use this for VBAT level Pyro"
-		(exclude_from_sim no)
-		(at 214.63 17.272 0)
-		(effects
-			(font
-				(size 1.27 1.27)
-			)
-		)
-	)
-	(text "Pyro Channels"
-		(exclude_from_sim no)
-		(at 182.626 14.224 0)
-		(effects
-			(font
-				(size 1.27 1.27)
-			)
-		)
-	)
-	(text "SSM3J328R PMOS\n"
-		(exclude_from_sim no)
-		(at 181.864 24.892 0)
-		(effects
-			(font
-				(size 1.27 1.27)
-			)
-		)
-	)
-	(text "5v Switching Regulator"
-		(exclude_from_sim no)
-		(at 40.386 124.206 0)
-		(effects
-			(font
-				(size 2.032 2.032)
-			)
-		)
-	)
-	(text "Global Current Sensing\n"
-		(exclude_from_sim no)
-		(at 140.97 78.232 0)
-		(effects
-			(font
-				(size 2.032 2.032)
-			)
-		)
-	)
-	(text "Need to implement two regs, 3.3v and 5v to run off of 2-3s lipo."
-		(exclude_from_sim no)
-		(at 56.388 48.006 0)
-		(effects
-			(font
-				(size 1.27 1.27)
-			)
-		)
-	)
-	(text "TODO: ensure all parts here are rated for voltage/amperage"
-		(exclude_from_sim no)
-		(at 96.012 130.048 0)
-		(effects
-			(font
-				(size 1.27 1.27)
-			)
-		)
-	)
-	(text "3.3v Switching Regulator\n"
-		(exclude_from_sim no)
-		(at 40.64 78.232 0)
-		(effects
-			(font
-				(size 2.032 2.032)
-			)
-		)
-	)
 	(global_label "FB"
 		(shape input)
@@
 		(shape input)
 		(at 242.57 48.26 180)
-		(fields_autoplaced yes)
 		(effects
 			(font
@@
 		(shape input)
 		(at 199.39 95.25 180)
-		(fields_autoplaced yes)
 		(effects
 			(font
@@
 		(shape input)
 		(at 243.84 96.52 180)
-		(fields_autoplaced yes)
 		(effects
 			(font
@@
 		(shape input)
 		(at 199.39 46.99 180)
-		(fields_autoplaced yes)
 		(effects
 			(font
@@
 		)
 	)
+	(sheet
+		(at 125.73 87.63)
+		(size 31.75 25.4)
+		(exclude_from_sim no)
+		(in_bom yes)
+		(on_board yes)
+		(dnp no)
+		(fields_autoplaced yes)
+		(stroke
+			(width 0.1524)
+			(type solid)
+		)
+		(fill
+			(color 0 0 0 0.0000)
+		)
+		(property "Sheetname" "Current Sense"
+			(at 125.73 86.9184 0)
+			(effects
+				(font
+					(size 1.27 1.27)
+				)
+				(justify left bottom)
+			)
+		)
+		(property "Sheetfile" "current_sense.kicad_sch"
+			(at 125.73 113.6146 0)
+			(effects
+				(font
+					(size 1.27 1.27)
+				)
+				(justify left top)
+			)
+		)
+		(instances
+			(project "NDXPPOWER"
+				(path "/1ee7f233-f9b1-483d-87ec-2f147a4d8262"
+					(page "2")
+				)
+			)
+		)
+	)
 	(sheet_instances
 		(path "/"
@@
 		)
 	)
+	(embedded_fonts no)
 )
