File: Power-Pyro/NDXPPOWER.kicad_sch (KiCad schematic)
At the start: 43 parts, among them J1 Conn_01x02, J5 Conn_01x02, J6 Conn_01x02, J7 Conn_01x02, Q1 SSM3J328R, Q2 SSM3J328R, Q3 L2N7002SLLT1G, Q4 L2N7002SLLT1G, Q5 SSM3J328R, Q6 SSM3J328R, Q7 L2N7002SLLT1G, Q8 L2N7002SLLT1G, U7 AP63203WU

Commit message: refactor🧮
Parts:
- removed C16, C19, C20, C21, C25, C26, C27, C28: 22uF, Capacitor_SMD:C_1206_3216Metric, symbol Device:C
- removed C18, C23: 100nF, Capacitor_SMD:C_0402_1005Metric, symbol Device:C
- removed C22: 2.2uF, Capacitor_SMD:C_0603_1608Metric, symbol Device:C
- removed C24: 470pF, Capacitor_SMD:C_0402_1005Metric, symbol Device:C
- removed J5, J6, J7: Conn_01x02, symbol Connector_Generic:Conn_01x02
- removed R13, R14, R15, R16: 100k, Resistor_SMD:R_0603_1608Metric, symbol Device:R
- removed R17: R, symbol Device:R
- removed U7: AP63203WU, Package_TO_SOT_SMD:TSOT-23-6, symbol Regulator_Switching:AP63203WU
- added C1: 10uF, Capacitor_SMD:C_0805_2012Metric, symbol Device:C
- added C10, C11, C12, C3, C6, C8, C9: 22uF, Capacitor_SMD:C_1206_3216Metric, symbol Device:C
- added C2: 470pF, Capacitor_SMD:C_0402_1005Metric, symbol Device:C
- added C4, C5: 100nF, Capacitor_SMD:C_0402_1005Metric, symbol Device:C
- added C7: 2.2uF, Capacitor_SMD:C_0603_1608Metric, symbol Device:C
- added J2, J3, J4: Conn_01x02, symbol Connector_Generic:Conn_01x02
- added R1: 1k, Resistor_SMD:R_0402_1005Metric, symbol Device:R
- added R2: 0, symbol Device:R
- added R3, R6, R7: 100k, Resistor_SMD:R_0603_1608Metric, symbol Device:R
- added U1: AP63203WU, Package_TO_SOT_SMD:TSOT-23-6, symbol Regulator_Switching:AP63203WU
- C13: value 10uF -> 22uF; footprint Capacitor_SMD:C_0805_2012Metric -> Capacitor_SMD:C_1206_3216Metric
- R11: value 0 -> 100k; footprint (none) -> Resistor_SMD:R_0603_1608Metric
- R12: value 1k -> 100k; footprint Resistor_SMD:R_0402_1005Metric -> Resistor_SMD:R_0603_1608Metric
- R4: value 100k -> R; footprint Resistor_SMD:R_0603_1608Metric -> (none)
Connections:
- net +3.3V: now also C3.1, C6.1, U1.1 (FB); no longer C15.1
- net +5V: now also C13.1, C15.1, R4.1, C11.1, C9.1
- net +BATT: now also C14.1, R10.1, R9.1, C1.1, C10.1, C12.1, C8.1, R6.1, U1.2 (EN), U1.3 (IN); no longer C13.1, R4.1
- net FB: now also C13.2, C15.2, R4.2, C11.2, C2.1, C9.2
- net GND: now also C14.2, C1.2, C10.2, C12.2, C3.2, C6.2, C7.1, C8.2, J2.1 (Pin_1), J3.1 (Pin_1), J4.1 (Pin_1), U1.4 (GND); no longer C13.2, C15.2
- net at L1.1: now also C4.1, U1.5 (SW); no longer C14.1
- net at Q8.1 (D): now also R12.2
- net at R9.2: now also Q5.2 (G), R11.1; no longer Q4.1 (D)
- net at Q6.1 (D): now also J4.2 (Pin_2)
- net at Q6.2 (G): now also R10.2, R12.1
- net at Q5.1 (D): now also J3.2 (Pin_2)
- net at PS1.10 (VCC): now also C7.2, R3.2; no longer R10.2
- net at L2.1, PS1.12 (SW), PS1.2 (SW): now also C5.2
- net at R11.2: now also Q7.1 (D); no longer PS1.13 (VBST)
- net at PS1.4 (PG): now also R3.1; no longer R10.1
- net at PS1.7 (FB): now also R1.2; no longer R12.2
- net at Q2.1 (D): now also J2.2 (Pin_2)
- net at Q3.1 (D): now also R7.2; no longer R8.2
- new net: C4.2, U1.6 (BST)
- new net: Q1.2 (G), R5.2, R7.1
- new net: PS1.13 (VBST), R2.2
- new net: Q2.2 (G), R6.2, R8.1
- new net: C2.2, R1.1
- new net: C5.1, R2.1
- new net: Q4.1 (D), R8.2

Commit message: terminal🚉
Parts:
- removed J4: Conn_01x02, symbol Connector_Generic:Conn_01x02
- added J5: Conn_01x02, TerminalBlock_Phoenix:TerminalBlock_Phoenix_MKDS-1,5-2-5.08_1x02_P5.08mm_Horizontal, symbol Connector_Generic:Conn_01x02
- J1, J2, J3: footprint (none) -> TerminalBlock_Phoenix:TerminalBlock_Phoenix_MKDS-1,5-2-5.08_1x02_P5.08mm_Horizontal
Connections:
- net GND: now also J5.1 (Pin_1)
- net at Q6.1 (D): now also J3.2 (Pin_2)
- net at Q5.1 (D): now also J5.2 (Pin_2); no longer J3.2 (Pin_2)
Changed lines of the file:
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@@
 			)
 		)
-		(property "Footprint" ""
+		(property "Footprint" "TerminalBlock_Phoenix:TerminalBlock_Phoenix_MKDS-1,5-2-5.08_1x02_P5.08mm_Horizontal"
 			(at 194.31 60.96 0)
 			(effects
@@
 	)
 	(symbol
+		(lib_id "Connector_Generic:Conn_01x02")
+		(at 237.49 62.23 270)
+		(unit 1)
+		(exclude_from_sim no)
+		(in_bom yes)
+		(on_board yes)
+		(dnp no)
+		(fields_autoplaced yes)
+		(property "Reference" "J5"
+			(at 240.03 60.9599 90)
+			(effects
+				(font
+					(size 1.27 1.27)
+				)
+				(justify left)
+			)
+		)
+		(property "Value" "Conn_01x02"
+			(at 240.03 63.4999 90)
+			(effects
+				(font
+					(size 1.27 1.27)
+				)
+				(justify left)
+			)
+		)
+		(property "Footprint" "TerminalBlock_Phoenix:TerminalBlock_Phoenix_MKDS-1,5-2-5.08_1x02_P5.08mm_Horizontal"
+			(at 237.49 62.23 0)
+			(effects
+				(font
+					(size 1.27 1.27)
+				)
+				(hide yes)
+			)
+		)
+		(property "Datasheet" "~"
+			(at 237.49 62.23 0)
+			(effects
+				(font
+					(size 1.27 1.27)
+				)
+				(hide yes)
+			)
+		)
+		(property "Description" "Generic connector, single row, 01x02, script generated (kicad-library-utils/schlib/autogen/connector/)"
+			(at 237.49 62.23 0)
+			(effects
+				(font
+					(size 1.27 1.27)
+				)
+				(hide yes)
+			)
+		)
+		(pin "2"
+		)
+		(pin "1"
+		)
+		(instances
+			(project "NDXPPOWER"
+				(path "/1ee7f233-f9b1-483d-87ec-2f147a4d8262"
+					(reference "J5")
+					(unit 1)
+				)
+			)
+		)
+	)
+	(symbol
 		(lib_id "Device:C")
 		(at 29.21 101.6 0)
@@
 		(dnp no)
 		(fields_autoplaced yes)
-		(property "Reference" "J4"
+		(property "Reference" "J3"
 			(at 241.3 109.2199 90)
 			(effects
@@
 			)
 		)
-		(property "Footprint" ""
+		(property "Footprint" "TerminalBlock_Phoenix:TerminalBlock_Phoenix_MKDS-1,5-2-5.08_1x02_P5.08mm_Horizontal"
 			(at 238.76 110.49 0)
 			(effects
@@
 			(project "NDXPPOWER"
 				(path "/1ee7f233-f9b1-483d-87ec-2f147a4d8262"
-					(reference "J4")
+					(reference "J3")
 					(unit 1)
 				)
@@
 	)
 	(symbol
-		(lib_id "Connector_Generic:Conn_01x02")
-		(at 237.49 62.23 270)
-		(unit 1)
-		(exclude_from_sim no)
-		(in_bom yes)
-		(on_board yes)
-		(dnp no)
-		(fields_autoplaced yes)
-		(property "Reference" "J3"
-			(at 240.03 60.9599 90)
-			(effects
-				(font
-					(size 1.27 1.27)
-				)
-				(justify left)
-			)
-		)
-		(property "Value" "Conn_01x02"
-			(at 240.03 63.4999 90)
-			(effects
-				(font
-					(size 1.27 1.27)
-				)
-				(justify left)
-			)
-		)
-		(property "Footprint" ""
-			(at 237.49 62.23 0)
-			(effects
-				(font
-					(size 1.27 1.27)
-				)
-				(hide yes)
-			)
-		)
-		(property "Datasheet" "~"
-			(at 237.49 62.23 0)
-			(effects
-				(font
-					(size 1.27 1.27)
-				)
-				(hide yes)
-			)
-		)
-		(property "Description" "Generic connector, single row, 01x02, script generated (kicad-library-utils/schlib/autogen/connector/)"
-			(at 237.49 62.23 0)
-			(effects
-				(font
-					(size 1.27 1.27)
-				)
-				(hide yes)
-			)
-		)
-		(pin "2"
-		)
-		(pin "1"
-		)
-		(instances
-			(project "NDXPPOWER"
-				(path "/1ee7f233-f9b1-483d-87ec-2f147a4d8262"
-					(reference "J3")
-					(unit 1)
-				)
-			)
-		)
-	)
-	(symbol
 		(lib_id "Device:R")
 		(at 114.3 170.18 0)
@@
 	)
 	(symbol
-		(lib_id "Connector_Generic:Conn_01x02")
-		(at 194.31 109.22 270)
-		(unit 1)
-		(exclude_from_sim no)
-		(in_bom yes)
-		(on_board yes)
-		(dnp no)
-		(fields_autoplaced yes)
-		(property "Reference" "J2"
-			(at 196.85 107.9499 90)
-			(effects
-				(font
-					(size 1.27 1.27)
-				)
-				(justify left)
-			)
-		)
-		(property "Value" "Conn_01x02"
-			(at 196.85 110.4899 90)
-			(effects
-				(font
-					(size 1.27 1.27)
-				)
-				(justify left)
-			)
-		)
-		(property "Footprint" ""
-			(at 194.31 109.22 0)
-			(effects
-				(font
-					(size 1.27 1.27)
-				)
-				(hide yes)
-			)
-		)
-		(property "Datasheet" "~"
-			(at 194.31 109.22 0)
-			(effects
-				(font
-					(size 1.27 1.27)
-				)
-				(hide yes)
-			)
-		)
-		(property "Description" "Generic connector, single row, 01x02, script generated (kicad-library-utils/schlib/autogen/connector/)"
-			(at 194.31 109.22 0)
-			(effects
-				(font
-					(size 1.27 1.27)
-				)
-				(hide yes)
-			)
-		)
-		(pin "2"
-		)
-		(pin "1"
-		)
-		(instances
-			(project "NDXPPOWER"
-				(path "/1ee7f233-f9b1-483d-87ec-2f147a4d8262"
-					(reference "J2")
-					(unit 1)
-				)
-			)
-		)
-	)
-	(symbol
 		(lib_id "Device:R")
 		(at 243.84 78.74 0)
@@
 					(unit 1)
 				)
+			)
+		)
+	)
+	(symbol
+		(lib_id "Connector_Generic:Conn_01x02")
+		(at 194.31 109.22 270)
+		(unit 1)
+		(exclude_from_sim no)
+		(in_bom yes)
+		(on_board yes)
+		(dnp no)
+		(fields_autoplaced yes)
+		(property "Reference" "J2"
+			(at 196.85 107.9499 90)
+			(effects
+				(font
+					(size 1.27 1.27)
+				)
+				(justify left)
+			)
+		)
+		(property "Value" "Conn_01x02"
+			(at 196.85 110.4899 90)
+			(effects
+				(font
+					(size 1.27 1.27)
+				)
+				(justify left)
+			)
+		)
+		(property "Footprint" "TerminalBlock_Phoenix:TerminalBlock_Phoenix_MKDS-1,5-2-5.08_1x02_P5.08mm_Horizontal"
+			(at 194.31 109.22 0)
+			(effects
+				(font
+					(size 1.27 1.27)
+				)
+				(hide yes)
+			)
+		)
+		(property "Datasheet" "~"
+			(at 194.31 109.22 0)
+			(effects
+				(font
+					(size 1.27 1.27)
+				)
+				(hide yes)
+			)
+		)
+		(property "Description" "Generic connector, single row, 01x02, script generated (kicad-library-utils/schlib/autogen/connector/)"
+			(at 194.31 109.22 0)
+			(effects
+				(font
+					(size 1.27 1.27)
+				)
+				(hide yes)
+			)
+		)
+		(pin "2"
+		)
+		(pin "1"
+		)
+		(instances
+			(project "NDXPPOWER"
+				(path "/1ee7f233-f9b1-483d-87ec-2f147a4d8262"
+					(reference "J2")
+					(unit 1)
+				)

Commit message: sd♠️
Parts:
- added H1, H2, H3, H4: MountingHole, MountingHole:MountingHole_2.2mm_M2_DIN965_Pad, symbol Mechanical:MountingHole

Commit message: refactor✖️
Parts:
- removed C1: 10uF, Capacitor_SMD:C_0805_2012Metric, symbol Device:C
- removed C10, C11, C12, C13, C15, C3, C6, C8, C9: 22uF, Capacitor_SMD:C_1206_3216Metric, symbol Device:C
- removed C14, C4, C5: 100nF, Capacitor_SMD:C_0402_1005Metric, symbol Device:C
- removed C2: 470pF, Capacitor_SMD:C_0402_1005Metric, symbol Device:C
- removed C7: 2.2uF, Capacitor_SMD:C_0603_1608Metric, symbol Device:C
- removed H1, H2, H3, H4: MountingHole, MountingHole:MountingHole_2.2mm_M2_DIN965_Pad, symbol Mechanical:MountingHole
- removed J1, J2, J3, J5: Conn_01x02, TerminalBlock_Phoenix:TerminalBlock_Phoenix_MKDS-1,5-2-5.08_1x02_P5.08mm_Horizontal, symbol Connector_Generic:Conn_01x02
- removed L1: 4.7uH, Inductor_SMD:L_1008_2520Metric, symbol Device:L
- removed L2: 1.5uH, Inductor_SMD:L_1008_2520Metric, symbol Device:L
- removed PS1: TPS513885VABR, TPS513885VABR:CONV_TPS513885VABR, symbol TPS513885VABR:TPS513885VABR
- removed Q1, Q2, Q5, Q6: SSM3J328R, SSM3J328R:SOT95P240X88-3N, symbol Simulation_SPICE:PMOS
- removed Q3, Q4, Q7, Q8: L2N7002SLLT1G, Package_TO_SOT_SMD:SOT-23, symbol Simulation_SPICE:NMOS
- removed R1: 1k, Resistor_SMD:R_0402_1005Metric, symbol Device:R
- removed R10, R11, R12, R3, R5, R6, R7, R8, R9: 100k, Resistor_SMD:R_0603_1608Metric, symbol Device:R
- removed R2: 0, symbol Device:R
- removed R4: R, symbol Device:R
- removed U1: AP63203WU, Package_TO_SOT_SMD:TSOT-23-6, symbol Regulator_Switching:AP63203WU
Connections:
- no-connect marks 1 -> 0
Other:
- added sheet 3.3vREG (3.3vREG.kicad_sch)
- added sheet 5vREG (5vREG.kicad_sch)
- added sheet CurrentSense (CurrentSense.kicad_sch)
- added sheet Peripherals (Peripherals.kicad_sch)
- added sheet Pyro (Pyro.kicad_sch)
- note added: "Running off 2-4S Lipo. 3.3v Regulator 5v Regulator current sensing ICs Resettable fuses on Pyro Channels"
- note removed: "3.3v Switching Regulator"
- note removed: "5v Switching Regulator"
- note removed: "Found this pmos by digikey, 20v, in stock, pmos, scrolling for high amperage"
- note removed: "From MCU USB port connected with diode"
- note removed: "Global Current Sensing"
- note removed: "Need to implement two regs, 3.3v and 5v to run off of 2-3s lipo."
- note removed: "Pyro Channels"
- note removed: "SSM3J328R PMOS"
- note removed: "TODO: ensure all parts here are rated for voltage/amperage"
- note removed: "Use this for VBAT level Pyro"

Commit message: 🔌
Other:
- note added: "Running off 2-4S Lipo. 3.3v Regulator 5v Regulator current sensing ICs Resettable fuses on Pyro Channels cool leds for pyto and whatnot"
- note removed: "Running off 2-4S Lipo. 3.3v Regulator 5v Regulator current sensing ICs Resettable fuses on Pyro Channels"
Changed lines of the file:
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@@
 		)
 	)
-	(text "Running off 2-4S Lipo.\n3.3v Regulator\n5v Regulator\ncurrent sensing ICs\nResettable fuses on Pyro Channels"
+	(text "Running off 2-4S Lipo.\n3.3v Regulator\n5v Regulator\ncurrent sensing ICs\nResettable fuses on Pyro Channels\ncool leds for pyto and whatnot\n"
 		(exclude_from_sim no)
 		(at 35.306 31.496 0)
