File: Power-Pyro/CurrentSense.kicad_sch (KiCad schematic)
At the start: 0 parts

Commit message: added current chip
Parts:
- added U2: INA260, Package_SO:TSSOP-16_4.4x5mm_P0.65mm, symbol Sensor:INA260
Connections:
- new net: U2.1 (IN+), U2.2 (IN+), U2.3 (IN+)
- new net: U2.11 (GND), U2.6 (GND)
- new net: U2.14 (IN-), U2.15 (IN-), U2.16 (IN-)
Changed lines of the file:
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@@
 (kicad_sch
-	(version 20231120)
+	(version 20250114)
 	(generator "eeschema")
-	(generator_version "8.0")
+	(generator_version "9.0")
 	(paper "A4")
+	(symbol
+		(lib_id "Sensor:INA260")
+		(at 143.51 87.63 0)
+		(unit 1)
+		(exclude_from_sim no)
+		(in_bom yes)
+		(on_board yes)
+		(dnp no)
+		(fields_autoplaced yes)
+		(property "Reference" "U2"
+			(at 145.6533 74.93 0)
+			(effects
+				(font
+					(size 1.27 1.27)
+				)
+				(justify left)
+			)
+		)
+		(property "Value" "INA260"
+			(at 145.6533 77.47 0)
+			(effects
+				(font
+					(size 1.27 1.27)
+				)
+				(justify left)
+			)
+		)
+		(property "Footprint" "Package_SO:TSSOP-16_4.4x5mm_P0.65mm"
+			(at 143.51 102.87 0)
+			(effects
+				(font
+					(size 1.27 1.27)
+				)
+				(hide yes)
+			)
+		)
+		(property "Datasheet" "http://www.ti.com/lit/ds/symlink/ina260.pdf"
+			(at 143.51 90.17 0)
+			(effects
+				(font
+					(size 1.27 1.27)
+				)
+				(hide yes)
+			)
+		)
+		(property "Description" "Current/power/voltage monitor with Integrated 2mΩ Shunt Resistor, 2.7V - 5.5V, I2C, TSSOP-16"
+			(at 143.51 87.63 0)
+			(effects
+				(font
+					(size 1.27 1.27)
+				)
+				(hide yes)
+			)
+		)
+		(pin "4"
+		)
+		(pin "5"
+		)
+		(pin "9"
+		)
+		(pin "8"
+		)
+		(pin "10"
+		)
+		(pin "3"
+		)
+		(pin "14"
+		)
+		(pin "12"
+		)
+		(pin "1"
+		)
+		(pin "15"
+		)
+		(pin "16"
+		)
+		(pin "13"
+		)
+		(pin "11"
+		)
+		(pin "6"
+		)
+		(pin "7"
+		)
+		(pin "2"
+		)
+		(instances
+			(project ""
+				(path "/1ee7f233-f9b1-483d-87ec-2f147a4d8262/d97e4bda-e8b9-4c0c-8657-284c28bc8cbd"
+					(reference "U2")
+					(unit 1)
+				)
+			)
+		)
+	)
 )
