File: Power-Pyro/NDXPPOWER.kicad_pcb (KiCad board)
At the start: 2 copper layers, 41 parts, among them J1 Conn_01x02, J2 Conn_01x02, J3 Conn_01x02, J5 Conn_01x02, Q1 SSM3J328R, Q2 SSM3J328R, Q3 L2N7002SLLT1G, Q4 L2N7002SLLT1G, Q5 SSM3J328R, Q6 SSM3J328R, Q7 L2N7002SLLT1G, Q8 L2N7002SLLT1G, U1 AP63203WU

Commit message: sd♠️
Parts:
- added H1: MountingHole, MountingHole:MountingHole_2.2mm_M2_DIN965_Pad, F.Cu at (129.6, 73.4)
- added H2: MountingHole, MountingHole:MountingHole_2.2mm_M2_DIN965_Pad, F.Cu at (154.1, 73.4)
- added H3: MountingHole, MountingHole:MountingHole_2.2mm_M2_DIN965_Pad, F.Cu at (129.6, 121.9)
- added H4: MountingHole, MountingHole:MountingHole_2.2mm_M2_DIN965_Pad, F.Cu at (154.1, 121.9)
- moved C10 60.5 mm to (74.1, 98.7)
- moved C11 60.5 mm to (74.1, 102.0)
- moved C12 60.5 mm to (74.1, 105.4)
- moved C13 60.5 mm to (74.1, 108.7)
- moved C14 60.5 mm to (86.3, 90.5)
- moved C15 60.5 mm to (74.1, 112.1)
- moved C2 60.5 mm to (86.3, 84.6)
- moved C3 60.5 mm to (74.1, 85.3)
- moved C4 60.5 mm to (86.3, 86.6)
- moved C5 60.5 mm to (86.3, 88.5)
- moved C6 60.5 mm to (74.1, 88.6)
- moved C8 60.5 mm to (74.1, 92.0)
- moved C9 60.5 mm to (74.1, 95.3)
- moved L1 60.5 mm to (89.4, 98.0)
- moved L2 60.5 mm to (89.4, 101.8)
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Other:
- board outline added: 31.5 x 55.5 mm

Commit message: FERBBBB🟣
Parts:
- added J4: Conn_01x02, TerminalBlock_Phoenix:TerminalBlock_Phoenix_MKDS-1,5-2-5.08_1x02_P5.08mm_Horizontal, F.Cu at (33.2, 92.5)
- J5: value Conn_01x02 -> Conn_02x06_Odd_Even; footprint TerminalBlock_Phoenix:TerminalBlock_Phoenix_MKDS-1,5-2-5.08_1x02_P5.08mm_Horizontal -> Connector_PinSocket_2.54mm:PinSocket_2x06_P2.54mm_Vertical_SMD
- moved J5 69.0 mm to (131.3, 101.0), turned to 0 degrees
Connections:
- net /PYRO_1 renamed /Pyro/PYRO_1
- net /PYRO_2 renamed /Pyro/PYRO_2
- net /PYRO_3 renamed /Pyro/PYRO_3
- net /PYRO_4 renamed /Pyro/PYRO_4
- C11 pad 1: USB_VBUS -> +5V
- C13 pad 1: USB_VBUS -> +5V
- C15 pad 1: USB_VBUS -> +5V
- C9 pad 1: USB_VBUS -> +5V
- J5 pad 1: GND -> /Peripherals/PYRO_1
- J5 pad 2: Net-(J5-Pin_2) -> unconnected-(J5-Pin_2-Pad2)
- L2 pad 2: USB_VBUS -> +5V
- Q5 pad 1: Net-(J5-Pin_2) -> Net-(J3-Pin_2)
- Q6 pad 1: Net-(J3-Pin_2) -> Net-(J4-Pin_2)

Commit message: 🔌
Parts:
- moved J5 2.20 mm to (131.2, 103.2)
Changed lines of the file:
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@@
 	(footprint "Connector_PinSocket_2.54mm:PinSocket_2x06_P2.54mm_Vertical_SMD"
 		(layer "F.Cu")
-		(at 131.28 101.05)
+		(at 131.18 103.25)
 		(descr "surface-mounted straight socket strip, 2x06, 2.54mm pitch, double cols (from Kicad 4.0.7), script generated")
 		(tags "Surface mounted socket strip SMD 2x06 2.54mm double row")

Commit message: test
Parts:
- added U2: INA260, Package_SO:TSSOP-16_4.4x5mm_P0.65mm, F.Cu at (97.6, 93.7)
